File: Arduino/pcb/mcu.sch (KiCad schematic (older format))
At the start: 0 parts

Commit message: pcb: continue wiring / move parts to hierachival sheets
Parts:
- added C5, C6: 100nF, symbol Device:C
- added C7, C8: 22pF, symbol Device:C
- added J9: FTDI, Connector_PinHeader_2.54mm:PinHeader_1x06_P2.54mm_Vertical, symbol ftdi:FTDI
- added R10, R11, R12, R13, R14, R15: 4K7, symbol Device:R
- added R7, R8: 100R, symbol Device:R
- added R9: 10K, symbol Device:R
- added SW2: Reset Button, Buttons_Switches_THT:SW_PUSH_6mm, symbol floppyorgel-rescue:SW_Push_Dual-RESCUE-floppyorgel
- added U3: ATMEGA328P-AU, Housings_QFP:TQFP-32_7x7mm_Pitch0.8mm, symbol floppyorgel-rescue:ATMEGA328P-AU-atmel
- added Y1: 20 Mhz Crystal, Crystals:Crystal_HC49-4H_Vertical, symbol floppyorgel-rescue:Crystal-device
Connections:
- new net: C8.1, U3.8 ((PCINT7/XTAL2/TOSC2)PB7), Y1.1
- new net: C7.2, U3.7 ((PCINT6/XTAL1/TOSC1)PB6), Y1.2
- new net: C6.1, R9.2, SW2.1, U3.29 ((PCINT14/~RESET~)PC6)
- new net: J9.4 (Transmit), R8.1, U3.30 ((PCINT16/RXD)PD0)
- new net: J9.5 (Receive), R7.1, U3.31 ((PCINT17/TXD)PD1)
- new net: C6.2, J9.6 (Ready_to_send)
- new net: R10.1, SW2.2
- new net 5V_ISP: J9.3 (VCC)
- new net DIRECTION: U3.13 ((PCINT1/OC1A)PB1)
- new net DRIVE_SELECT: U3.12 ((PCINT0/CLKO/ICP1)PB0)
- new net GND: C5.2, C7.1, C8.2, J9.1 (Ground), R10.2, R11.1, R12.1, R13.1, R14.1, R15.1, U3.21 (GND), U3.3 (GND), U3.5 (GND)
- new net LATCH_ADDR: R11.2, U3.24 ((PCINT9/ADC1)PC1)
- new net LATCH_LED: R12.2, U3.25 ((PCINT10/ADC2)PC2)
- new net MISO: R13.2, U3.16 ((PCINT4/MISO)PB4)
- new net MOSI: R14.2, U3.15 ((PCINT3/OC2A/MOSI)PB3)
- new net RX: R8.2
- new net SCK: R15.2, U3.17 ((PCINT5/SCK)PB5)
- new net STEP: U3.14 ((PCINT2/OC1B/~SS~)PB2)
- new net TRK00: U3.23 ((PCINT8/ADC0)PC0)
- new net TX: R7.2
- new net VCC: C5.1, R9.1, U3.18 (AVCC), U3.4 (VCC), U3.6 (VCC)
- no-connect marks 0 -> 13
Other:
- note added: "Bypass"

Commit message: pcb: finish wiring / use ws2812 under chip led
Parts:
- removed R12, R14: 4K7, symbol Device:R
- renumbered C5 to C4, C6 to C5, C7 to C6, C8 to C7, R13 to R12, R15 to R13, U3 to U2
Connections:
- net LATCH_LED renamed DATA_LED
- net MOSI: no longer names the net of U2.15 ((PCINT3/OC2A/MOSI)PB3)
- no-connect marks 13 -> 14
Other:
- moved on the sheet: R12, R13
Changed lines of the file:
@@
 $Descr A4 11693 8268
 encoding utf-8
-Sheet 6 6
+Sheet 5 6
 Title ""
 Date ""
@@
 P 7050 3275
 AR Path="/5CC6665F" Ref="C?"  Part="1"
-AR Path="/5CCFEC3E/5CC6665F" Ref="C8"  Part="1"
-F 0 "C8" V 6800 3275 50  0000 C CNN
+AR Path="/5CCFEC3E/5CC6665F" Ref="C7"  Part="1"
+F 0 "C7" V 6800 3275 50  0000 C CNN
 F 1 "22pF" V 6900 3275 50  0000 C CNN
 F 2 "" H 7088 3125 50  0001 C CNN
@@
 P 7375 3275
 AR Path="/5CC66665" Ref="#PWR?"  Part="1"
-AR Path="/5CCFEC3E/5CC66665" Ref="#PWR030"  Part="1"
-F 0 "#PWR030" H 7375 3025 50  0001 C CNN
+AR Path="/5CCFEC3E/5CC66665" Ref="#PWR023"  Part="1"
+F 0 "#PWR023" H 7375 3025 50  0001 C CNN
 F 1 "GND" H 7380 3102 50  0000 C CNN
 F 2 "" H 7375 3275 50  0001 C CNN
@@
 P 7050 2975
 AR Path="/5CC6666B" Ref="C?"  Part="1"
-AR Path="/5CCFEC3E/5CC6666B" Ref="C7"  Part="1"
-F 0 "C7" V 6798 2975 50  0000 C CNN
+AR Path="/5CCFEC3E/5CC6666B" Ref="C6"  Part="1"
+F 0 "C6" V 6798 2975 50  0000 C CNN
 F 1 "22pF" V 6889 2975 50  0000 C CNN
 F 2 "" H 7088 2825 50  0001 C CNN
@@
 P 4825 3575
 AR Path="/5CC6668C" Ref="U?"  Part="1"
-AR Path="/5CCFEC3E/5CC6668C" Ref="U3"  Part="1"
-F 0 "U3" H 4075 4825 50  0000 L BNN
+AR Path="/5CCFEC3E/5CC6668C" Ref="U2"  Part="1"
+F 0 "U2" H 4075 4825 50  0000 L BNN
 F 1 "ATMEGA328P-AU" H 5225 2175 50  0000 L BNN
 F 2 "Housings_QFP:TQFP-32_7x7mm_Pitch0.8mm" H 4825 3575 50  0001 C CIN
@@
 Text HLabel 5875 2675 2    50   Output ~ 0
 STEP
-Text HLabel 5875 2775 2    50   Output ~ 0
-MOSI
 Text HLabel 5875 2875 2    50   Input ~ 0
 MISO
@@
 LATCH_ADDR
 Text HLabel 5875 3525 2    50   Output ~ 0
-LATCH_LED
+DATA_LED
 $Comp
 L ftdi:FTDI J9
@@
 $EndComp
 $Comp
-L power:GND #PWR031
+L power:GND #PWR024
 U 1 1 5CCD776A
 P 7400 5500
-F 0 "#PWR031" H 7400 5250 50  0001 C CNN
+F 0 "#PWR024" H 7400 5250 50  0001 C CNN
 F 1 "GND" H 7405 5327 50  0000 C CNN
 F 2 "" H 7400 5500 50  0001 C CNN
@@
 Connection ~ 7250 3925
 $Comp
-L power:GND #PWR032
+L power:GND #PWR025
 U 1 1 5CCED0DE
 P 8000 4525
-F 0 "#PWR032" H 8000 4275 50  0001 C CNN
+F 0 "#PWR025" H 8000 4275 50  0001 C CNN
 F 1 "GND" H 8005 4352 50  0000 C CNN
 F 2 "" H 8000 4525 50  0001 C CNN
@@
 $EndComp
 $Comp
-L power:VCC #PWR029
+L power:VCC #PWR022
 U 1 1 5CCED0EA
 P 6700 3525
-F 0 "#PWR029" H 6700 3375 50  0001 C CNN
+F 0 "#PWR022" H 6700 3375 50  0001 C CNN
 F 1 "VCC" H 6717 3698 50  0000 C CNN
 F 2 "" H 6700 3525 50  0001 C CNN
@@
 	7650 4025 8000 4025
 $Comp
-L Device:C C6
+L Device:C C5
 U 1 1 5CCED101
 P 6825 4200
-F 0 "C6" H 7025 4250 50  0000 L CNN
+F 0 "C5" H 7025 4250 50  0000 L CNN
 F 1 "100nF" H 6975 4150 50  0000 L CNN
 F 2 "" H 6863 4050 50  0001 C CNN
@@
 5V_ISP
 $Comp
-L power:VCC #PWR027
+L power:VCC #PWR020
 U 1 1 5CE9FC49
 P 3625 2475
-F 0 "#PWR027" H 3625 2325 50  0001 C CNN
+F 0 "#PWR020" H 3625 2325 50  0001 C CNN
 F 1 "VCC" H 3642 2648 50  0000 C CNN
 F 2 "" H 3625 2475 50  0001 C CNN
@@
 Connection ~ 3625 2475
 $Comp
-L power:GND #PWR028
+L power:GND #PWR021
 U 1 1 5CEA02DB
 P 3625 4775
-F 0 "#PWR028" H 3625 4525 50  0001 C CNN
+F 0 "#PWR021" H 3625 4525 50  0001 C CNN
 F 1 "GND" H 3630 4602 50  0000 C CNN
 F 2 "" H 3625 4775 50  0001 C CNN
@@
 P 3025 2700
 AR Path="/5D1392AB" Ref="C?"  Part="1"
-AR Path="/5CCFEC3E/5D1392AB" Ref="C5"  Part="1"
-F 0 "C5" H 2800 2900 50  0000 L CNN
+AR Path="/5CCFEC3E/5D1392AB" Ref="C4"  Part="1"
+F 0 "C4" H 2800 2900 50  0000 L CNN
 F 1 "100nF" H 2750 2800 50  0000 L CNN
 F 2 "" H 3063 2550 50  0001 C CNN
@@
 $EndComp
 $Comp
-L power:VCC #PWR025
+L power:VCC #PWR018
 U 1 1 5D13AC7F
 P 3025 2425
-F 0 "#PWR025" H 3025 2275 50  0001 C CNN
+F 0 "#PWR018" H 3025 2275 50  0001 C CNN
 F 1 "VCC" H 3042 2598 50  0000 C CNN
 F 2 "" H 3025 2425 50  0001 C CNN
@@
 $EndComp
 $Comp
-L power:GND #PWR026
+L power:GND #PWR019
 U 1 1 5D13B83C
 P 3025 2950
-F 0 "#PWR026" H 3025 2700 50  0001 C CNN
+F 0 "#PWR019" H 3025 2700 50  0001 C CNN
 F 1 "GND" H 3030 2777 50  0000 C CNN
 F 2 "" H 3025 2950 50  0001 C CNN
@@
 	8050 2500 8050 2600
 Wire Wire Line
+	8250 2500 8250 2600
+Wire Wire Line
 	8150 2500 8150 2600
 Wire Wire Line
-	8450 2500 8450 2600
-Wire Wire Line
-	8350 2500 8350 2600
-Wire Wire Line
-	8250 2500 8250 2600
-Connection ~ 8050 2900
-Wire Wire Line
-	8050 2900 8150 2900
-Wire Wire Line
 	8050 2900 8050 2950
-Connection ~ 8150 2900
-Connection ~ 8250 2900
-Wire Wire Line
-	8150 2900 8250 2900
-Wire Wire Line
-	8350 2900 8250 2900
-Connection ~ 8350 2900
-Wire Wire Line
-	8450 2900 8350 2900
 $Comp
 L power:GND #PWR?
@@
 P 8050 2950
 AR Path="/5D158700" Ref="#PWR?"  Part="1"
-AR Path="/5CCFEC3E/5D158700" Ref="#PWR033"  Part="1"
-F 0 "#PWR033" H 8050 2700 50  0001 C CNN
+AR Path="/5CCFEC3E/5D158700" Ref="#PWR026"  Part="1"
+F 0 "#PWR026" H 8050 2700 50  0001 C CNN
 F 1 "GND" H 8055 2777 50  0000 C CNN
 F 2 "" H 8050 2950 50  0001 C CNN
@@
 LATCH_ADDR
 Text HLabel 8150 2500 1    50   Input ~ 0
-LATCH_LED
+MISO
 Text HLabel 8250 2500 1    50   Input ~ 0
-MISO
-Text HLabel 8350 2500 1    50   Input ~ 0
-MOSI
-Text HLabel 8450 2500 1    50   Input ~ 0
 SCK
 $Comp
 L Device:R R?
 U 1 1 5D1586EE
-P 8450 2750
+P 8250 2750
 AR Path="/5D1586EE" Ref="R?"  Part="1"
-AR Path="/5CCFEC3E/5D1586EE" Ref="R15"  Part="1"
-F 0 "R15" V 8475 2575 50  0000 C CNN
-F 1 "4K7" V 8450 2750 50  0000 C CNN
-F 2 "" V 8380 2750 50  0001 C CNN
-F 3 "~" H 8450 2750 50  0001 C CNN
-	1    8450 2750
-	-1   0    0    1
-$EndComp
-$Comp
-L Device:R R?
-U 1 1 5D1586F4
-P 8350 2750
-AR Path="/5D1586F4" Ref="R?"  Part="1"
-AR Path="/5CCFEC3E/5D1586F4" Ref="R14"  Part="1"
-F 0 "R14" V 8375 2575 50  0000 C CNN
-F 1 "4K7" V 8350 2750 50  0000 C CNN
-F 2 "" V 8280 2750 50  0001 C CNN
-F 3 "~" H 8350 2750 50  0001 C CNN
-	1    8350 2750
-	-1   0    0    1
-$EndComp
-$Comp
-L Device:R R?
-U 1 1 5D1586FA
-P 8250 2750
-AR Path="/5D1586FA" Ref="R?"  Part="1"
-AR Path="/5CCFEC3E/5D1586FA" Ref="R13"  Part="1"
+AR Path="/5CCFEC3E/5D1586EE" Ref="R13"  Part="1"
 F 0 "R13" V 8275 2575 50  0000 C CNN
 F 1 "4K7" V 8250 2750 50  0000 C CNN
@@
 $Comp
 L Device:R R?
-U 1 1 5D1586E5
+U 1 1 5D1586FA
 P 8150 2750
-AR Path="/5D1586E5" Ref="R?"  Part="1"
-AR Path="/5CCFEC3E/5D1586E5" Ref="R12"  Part="1"
+AR Path="/5D1586FA" Ref="R?"  Part="1"
+AR Path="/5CCFEC3E/5D1586FA" Ref="R12"  Part="1"
 F 0 "R12" V 8175 2575 50  0000 C CNN
 F 1 "4K7" V 8150 2750 50  0000 C CNN
@@
 Wire Wire Line
 	6525 4450 6525 4550
+NoConn ~ 5875 2775
+Wire Wire Line
+	8250 2900 8150 2900
+Wire Wire Line
+	8150 2900 8050 2900
+Connection ~ 8150 2900
+Connection ~ 8050 2900
 $EndSCHEMATC

Commit message: pcb: assign footprints
Parts:
- C4, C5, C6, C7, R10, R11, R12, R13, R7, R8, R9: footprint (none) -> Capacitor_SMD:C_0201_0603Metric
- SW2: footprint Buttons_Switches_THT:SW_PUSH_6mm -> Button_Switch_THT:SW_PUSH_6mm
- U2: footprint Housings_QFP:TQFP-32_7x7mm_Pitch0.8mm -> Package_QFP:LQFP-32_7x7mm_P0.8mm
- Y1: footprint Crystals:Crystal_HC49-4H_Vertical -> Crystal:Crystal_HC49-4H_Vertical
Changed lines of the file:
@@
 F 0 "C7" V 6800 3275 50  0000 C CNN
 F 1 "22pF" V 6900 3275 50  0000 C CNN
-F 2 "" H 7088 3125 50  0001 C CNN
+F 2 "Capacitor_SMD:C_0201_0603Metric" H 7088 3125 50  0001 C CNN
 F 3 "~" H 7050 3275 50  0001 C CNN
 	1    7050 3275
@@
 F 0 "C6" V 6798 2975 50  0000 C CNN
 F 1 "22pF" V 6889 2975 50  0000 C CNN
-F 2 "" H 7088 2825 50  0001 C CNN
+F 2 "Capacitor_SMD:C_0201_0603Metric" H 7088 2825 50  0001 C CNN
 F 3 "~" H 7050 2975 50  0001 C CNN
 	1    7050 2975
@@
 F 0 "Y1" V 6975 3125 50  0000 C CNN
 F 1 "20 Mhz Crystal" V 6875 3125 50  0000 C CNN
-F 2 "Crystals:Crystal_HC49-4H_Vertical" H 6625 3125 50  0001 C CNN
+F 2 "Crystal:Crystal_HC49-4H_Vertical" H 6625 3125 50  0001 C CNN
 F 3 "" H 6625 3125 50  0001 C CNN
 	1    6625 3125
@@
 F 0 "U2" H 4075 4825 50  0000 L BNN
 F 1 "ATMEGA328P-AU" H 5225 2175 50  0000 L BNN
-F 2 "Housings_QFP:TQFP-32_7x7mm_Pitch0.8mm" H 4825 3575 50  0001 C CIN
+F 2 "Package_QFP:LQFP-32_7x7mm_P0.8mm" H 4825 3575 50  0001 C CIN
 F 3 "" H 4825 3575 50  0001 C CNN
 	1    4825 3575
@@
 F 0 "SW2" H 7500 3925 50  0000 L CNN
 F 1 "Reset Button" H 7450 3555 50  0000 C CNN
-F 2 "Buttons_Switches_THT:SW_PUSH_6mm" H 7450 4025 50  0001 C CNN
+F 2 "Button_Switch_THT:SW_PUSH_6mm" H 7450 4025 50  0001 C CNN
 F 3 "" H 7450 4025 50  0001 C CNN
 	1    7450 3825
@@
 F 0 "R9" H 6770 3721 50  0000 L CNN
 F 1 "10K" H 6770 3630 50  0000 L CNN
-F 2 "" V 6630 3675 50  0001 C CNN
+F 2 "Capacitor_SMD:C_0201_0603Metric" V 6630 3675 50  0001 C CNN
 F 3 "~" H 6700 3675 50  0001 C CNN
 	1    6700 3675
@@
 F 0 "C5" H 7025 4250 50  0000 L CNN
 F 1 "100nF" H 6975 4150 50  0000 L CNN
-F 2 "" H 6863 4050 50  0001 C CNN
+F 2 "Capacitor_SMD:C_0201_0603Metric" H 6863 4050 50  0001 C CNN
 F 3 "~" H 6825 4200 50  0001 C CNN
 	1    6825 4200
@@
 F 0 "R10" H 8070 4371 50  0000 L CNN
 F 1 "4K7" H 8070 4280 50  0000 L CNN
-F 2 "" V 7930 4325 50  0001 C CNN
+F 2 "Capacitor_SMD:C_0201_0603Metric" V 7930 4325 50  0001 C CNN
 F 3 "~" H 8000 4325 50  0001 C CNN
 	1    8000 4325
@@
 F 0 "R7" H 6275 4850 50  0000 L CNN
 F 1 "100R" V 6425 4600 50  0000 L CNN
-F 2 "" V 6355 4700 50  0001 C CNN
+F 2 "Capacitor_SMD:C_0201_0603Metric" V 6355 4700 50  0001 C CNN
 F 3 "~" H 6425 4700 50  0001 C CNN
 	1    6425 4700
@@
 F 0 "R8" H 6425 4850 50  0000 L CNN
 F 1 "100R" V 6525 4600 50  0000 L CNN
-F 2 "" V 6455 4700 50  0001 C CNN
+F 2 "Capacitor_SMD:C_0201_0603Metric" V 6455 4700 50  0001 C CNN
 F 3 "~" H 6525 4700 50  0001 C CNN
 	1    6525 4700
@@
 F 0 "C4" H 2800 2900 50  0000 L CNN
 F 1 "100nF" H 2750 2800 50  0000 L CNN
-F 2 "" H 3063 2550 50  0001 C CNN
+F 2 "Capacitor_SMD:C_0201_0603Metric" H 3063 2550 50  0001 C CNN
 F 3 "~" H 3025 2700 50  0001 C CNN
 	1    3025 2700
@@
 F 0 "R13" V 8275 2575 50  0000 C CNN
 F 1 "4K7" V 8250 2750 50  0000 C CNN
-F 2 "" V 8180 2750 50  0001 C CNN
+F 2 "Capacitor_SMD:C_0201_0603Metric" V 8180 2750 50  0001 C CNN
 F 3 "~" H 8250 2750 50  0001 C CNN
 	1    8250 2750
@@
 F 0 "R12" V 8175 2575 50  0000 C CNN
 F 1 "4K7" V 8150 2750 50  0000 C CNN
-F 2 "" V 8080 2750 50  0001 C CNN
+F 2 "Capacitor_SMD:C_0201_0603Metric" V 8080 2750 50  0001 C CNN
 F 3 "~" H 8150 2750 50  0001 C CNN
 	1    8150 2750
@@
 F 0 "R11" V 8075 2575 50  0000 C CNN
 F 1 "4K7" V 8050 2750 50  0000 C CNN
-F 2 "" V 7980 2750 50  0001 C CNN
+F 2 "Capacitor_SMD:C_0201_0603Metric" V 7980 2750 50  0001 C CNN
 F 3 "~" H 8050 2750 50  0001 C CNN
 	1    8050 2750

Commit message: pcb: add I2C eeprom
Parts:
- added U3: 24LC64, Package_SO:TSSOP-8_4.4x3mm_P0.65mm, symbol Memory_EEPROM:24LC64
- renumbered C4 to C3, C5 to C4, C6 to C5, C7 to C6
Connections:
- net GND: now also U3.1 (A0), U3.2 (A1), U3.3 (A2), U3.4 (GND), U3.7 (WP)
- net VCC: now also U3.8 (VCC)
- net SDA: now reaches U2.27 ((PCINT12/SDA/ADC4)PC4)
- net SDA: now also U3.5 (SDA)
- net SCL: now reaches U2.28 ((PCINT13/SCL/ADC5)PC5)
- net SCL: now also U3.6 (SCL)
- no-connect marks 14 -> 12
Changed lines of the file:
@@
 $EndDescr
 NoConn ~ 5825 3625
-NoConn ~ 5825 3725
-NoConn ~ 5825 3825
 NoConn ~ 5825 4775
 NoConn ~ 5825 4675
@@
 P 7050 3275
 AR Path="/5CC6665F" Ref="C?"  Part="1"
-AR Path="/5CCFEC3E/5CC6665F" Ref="C7"  Part="1"
-F 0 "C7" V 6800 3275 50  0000 C CNN
+AR Path="/5CCFEC3E/5CC6665F" Ref="C6"  Part="1"
+F 0 "C6" V 6800 3275 50  0000 C CNN
 F 1 "22pF" V 6900 3275 50  0000 C CNN
 F 2 "Capacitor_SMD:C_0201_0603Metric" H 7088 3125 50  0001 C CNN
@@
 P 7375 3275
 AR Path="/5CC66665" Ref="#PWR?"  Part="1"
-AR Path="/5CCFEC3E/5CC66665" Ref="#PWR023"  Part="1"
-F 0 "#PWR023" H 7375 3025 50  0001 C CNN
+AR Path="/5CCFEC3E/5CC66665" Ref="#PWR022"  Part="1"
+F 0 "#PWR022" H 7375 3025 50  0001 C CNN
 F 1 "GND" H 7380 3102 50  0000 C CNN
 F 2 "" H 7375 3275 50  0001 C CNN
@@
 P 7050 2975
 AR Path="/5CC6666B" Ref="C?"  Part="1"
-AR Path="/5CCFEC3E/5CC6666B" Ref="C6"  Part="1"
-F 0 "C6" V 6798 2975 50  0000 C CNN
+AR Path="/5CCFEC3E/5CC6666B" Ref="C5"  Part="1"
+F 0 "C5" V 6798 2975 50  0000 C CNN
 F 1 "22pF" V 6889 2975 50  0000 C CNN
 F 2 "Capacitor_SMD:C_0201_0603Metric" H 7088 2825 50  0001 C CNN
@@
 $EndComp
 $Comp
-L power:GND #PWR024
+L power:GND #PWR023
 U 1 1 5CCD776A
 P 7400 5500
-F 0 "#PWR024" H 7400 5250 50  0001 C CNN
+F 0 "#PWR023" H 7400 5250 50  0001 C CNN
 F 1 "GND" H 7405 5327 50  0000 C CNN
 F 2 "" H 7400 5500 50  0001 C CNN
@@
 Connection ~ 7250 3925
 $Comp
-L power:GND #PWR025
+L power:GND #PWR024
 U 1 1 5CCED0DE
 P 8000 4525
-F 0 "#PWR025" H 8000 4275 50  0001 C CNN
+F 0 "#PWR024" H 8000 4275 50  0001 C CNN
 F 1 "GND" H 8005 4352 50  0000 C CNN
 F 2 "" H 8000 4525 50  0001 C CNN
@@
 $EndComp
 $Comp
-L power:VCC #PWR022
+L power:VCC #PWR021
 U 1 1 5CCED0EA
 P 6700 3525
-F 0 "#PWR022" H 6700 3375 50  0001 C CNN
+F 0 "#PWR021" H 6700 3375 50  0001 C CNN
 F 1 "VCC" H 6717 3698 50  0000 C CNN
 F 2 "" H 6700 3525 50  0001 C CNN
@@
 	7650 4025 8000 4025
 $Comp
-L Device:C C5
+L Device:C C4
 U 1 1 5CCED101
 P 6825 4200
-F 0 "C5" H 7025 4250 50  0000 L CNN
+F 0 "C4" H 7025 4250 50  0000 L CNN
 F 1 "100nF" H 6975 4150 50  0000 L CNN
 F 2 "Capacitor_SMD:C_0201_0603Metric" H 6863 4050 50  0001 C CNN
@@
 5V_ISP
 $Comp
-L power:VCC #PWR020
+L power:VCC #PWR019
 U 1 1 5CE9FC49
 P 3625 2475
-F 0 "#PWR020" H 3625 2325 50  0001 C CNN
+F 0 "#PWR019" H 3625 2325 50  0001 C CNN
 F 1 "VCC" H 3642 2648 50  0000 C CNN
 F 2 "" H 3625 2475 50  0001 C CNN
@@
 Connection ~ 3625 2475
 $Comp
-L power:GND #PWR021
+L power:GND #PWR020
 U 1 1 5CEA02DB
 P 3625 4775
-F 0 "#PWR021" H 3625 4525 50  0001 C CNN
+F 0 "#PWR020" H 3625 4525 50  0001 C CNN
 F 1 "GND" H 3630 4602 50  0000 C CNN
 F 2 "" H 3625 4775 50  0001 C CNN
@@
 P 3025 2700
 AR Path="/5D1392AB" Ref="C?"  Part="1"
-AR Path="/5CCFEC3E/5D1392AB" Ref="C4"  Part="1"
-F 0 "C4" H 2800 2900 50  0000 L CNN
+AR Path="/5CCFEC3E/5D1392AB" Ref="C3"  Part="1"
+F 0 "C3" H 2800 2900 50  0000 L CNN
 F 1 "100nF" H 2750 2800 50  0000 L CNN
 F 2 "Capacitor_SMD:C_0201_0603Metric" H 3063 2550 50  0001 C CNN
@@
 $EndComp
 $Comp
-L power:VCC #PWR018
+L power:VCC #PWR017
 U 1 1 5D13AC7F
 P 3025 2425
-F 0 "#PWR018" H 3025 2275 50  0001 C CNN
+F 0 "#PWR017" H 3025 2275 50  0001 C CNN
 F 1 "VCC" H 3042 2598 50  0000 C CNN
 F 2 "" H 3025 2425 50  0001 C CNN
@@
 $EndComp
 $Comp
-L power:GND #PWR019
+L power:GND #PWR018
 U 1 1 5D13B83C
 P 3025 2950
-F 0 "#PWR019" H 3025 2700 50  0001 C CNN
+F 0 "#PWR018" H 3025 2700 50  0001 C CNN
 F 1 "GND" H 3030 2777 50  0000 C CNN
 F 2 "" H 3025 2950 50  0001 C CNN
@@
 P 8050 2950
 AR Path="/5D158700" Ref="#PWR?"  Part="1"
-AR Path="/5CCFEC3E/5D158700" Ref="#PWR026"  Part="1"
-F 0 "#PWR026" H 8050 2700 50  0001 C CNN
+AR Path="/5CCFEC3E/5D158700" Ref="#PWR025"  Part="1"
+F 0 "#PWR025" H 8050 2700 50  0001 C CNN
 F 1 "GND" H 8055 2777 50  0000 C CNN
 F 2 "" H 8050 2950 50  0001 C CNN
@@
 Connection ~ 8150 2900
 Connection ~ 8050 2900
+$Comp
+L Memory_EEPROM:24LC64 U3
+U 1 1 5CCCB27C
+P 9075 3650
+F 0 "U3" H 8850 4050 50  0000 C CNN
+F 1 "24LC64" H 8850 3950 50  0000 C CNN
+F 2 "Package_SO:TSSOP-8_4.4x3mm_P0.65mm" H 9075 3650 50  0001 C CNN
+F 3 "http://ww1.microchip.com/downloads/en/DeviceDoc/21189f.pdf" H 9075 3650 50  0001 C CNN
+	1    9075 3650
+	-1   0    0    -1
+$EndComp
+Text Label 5925 3725 0    50   ~ 0
+SDA
+Text Label 5925 3825 0    50   ~ 0
+SCL
+Wire Wire Line
+	5825 3725 5925 3725
+Wire Wire Line
+	5825 3825 5925 3825
+Text Label 8575 3550 2    50   ~ 0
+SDA
+Text Label 8575 3650 2    50   ~ 0
+SCL
+Wire Wire Line
+	8575 3550 8675 3550
+Wire Wire Line
+	8575 3650 8675 3650
+$Comp
+L power:VCC #PWR027
+U 1 1 5CCEB8A8
+P 9075 3250
+F 0 "#PWR027" H 9075 3100 50  0001 C CNN
+F 1 "VCC" H 9092 3423 50  0000 C CNN
+F 2 "" H 9075 3250 50  0001 C CNN
+F 3 "" H 9075 3250 50  0001 C CNN
+	1    9075 3250
+	1    0    0    -1
+$EndComp
+$Comp
+L power:GND #PWR028
+U 1 1 5CCEC3F1
+P 9075 4050
+F 0 "#PWR028" H 9075 3800 50  0001 C CNN
+F 1 "GND" H 9080 3877 50  0000 C CNN
+F 2 "" H 9075 4050 50  0001 C CNN
+F 3 "" H 9075 4050 50  0001 C CNN
+	1    9075 4050
+	1    0    0    -1
+$EndComp
+Wire Wire Line
+	9075 3350 9075 3250
+Wire Wire Line
+	9075 3950 9075 4050
+Wire Wire Line
+	9475 3750 9575 3750
+Wire Wire Line
+	9475 3650 9575 3650
+Wire Wire Line
+	9575 3650 9575 3750
+Wire Wire Line
+	9475 3550 9575 3550
+Wire Wire Line
+	9575 3550 9575 3650
+Connection ~ 9575 3650
+$Comp
+L power:GND #PWR029
+U 1 1 5CD0D0C1
+P 9575 4050
+F 0 "#PWR029" H 9575 3800 50  0001 C CNN
+F 1 "GND" H 9580 3877 50  0000 C CNN
+F 2 "" H 9575 4050 50  0001 C CNN
+F 3 "" H 9575 4050 50  0001 C CNN
+	1    9575 4050
+	1    0    0    -1
+$EndComp
+Wire Wire Line
+	9575 3750 9575 4050
+Connection ~ 9575 3750
+$Comp
+L power:GND #PWR026
+U 1 1 5CD10438
+P 8575 4050
+F 0 "#PWR026" H 8575 3800 50  0001 C CNN
+F 1 "GND" H 8580 3877 50  0000 C CNN
+F 2 "" H 8575 4050 50  0001 C CNN
+F 3 "" H 8575 4050 50  0001 C CNN
+	1    8575 4050
+	1    0    0    -1
+$EndComp
+Wire Wire Line
+	8675 3750 8575 3750
+Wire Wire Line
+	8575 3750 8575 4050
 $EndSCHEMATC
