File: Arduino/pcb/mcu.sch (KiCad schematic (older format))
At the start: 16 parts, among them J9 FTDI, SW2 Reset Button, U2 ATMEGA328P-AU, U3 24LC64, Y1 20 Mhz Crystal

Commit message: pcb: continue placement + add some info on silk
Parts:
- added C7: 100nF, Capacitor_SMD:C_0805_2012Metric, symbol Device:C
- C3: renamed from C4; footprint Capacitor_SMD:C_0201_0603Metric -> Capacitor_SMD:C_0805_2012Metric
- C4: renamed from C5; footprint Capacitor_SMD:C_0201_0603Metric -> Capacitor_SMD:C_0805_2012Metric
- C5: renamed from C6; footprint Capacitor_SMD:C_0201_0603Metric -> Capacitor_SMD:C_0805_2012Metric
- C6: renamed from C3; footprint Capacitor_SMD:C_0201_0603Metric -> Capacitor_SMD:C_0805_2012Metric
- R10, R11, R12, R13, R7, R8, R9: footprint Capacitor_SMD:C_0201_0603Metric -> Resistor_SMD:R_0805_2012Metric
Connections:
- net GND: now also C7.2
- net VCC: now also C7.1
- net MOSI: now reaches U2.15 ((PCINT3/OC2A/MOSI)PB3)
- net DATA_LED renamed LATCH_LED
- no-connect marks 12 -> 11
Other:
- moved on the sheet: C6
Changed lines of the file:
@@
 P 7050 3275
 AR Path="/5CC6665F" Ref="C?"  Part="1"
-AR Path="/5CCFEC3E/5CC6665F" Ref="C6"  Part="1"
-F 0 "C6" V 6800 3275 50  0000 C CNN
+AR Path="/5CCFEC3E/5CC6665F" Ref="C5"  Part="1"
+F 0 "C5" V 6800 3275 50  0000 C CNN
 F 1 "22pF" V 6900 3275 50  0000 C CNN
-F 2 "Capacitor_SMD:C_0201_0603Metric" H 7088 3125 50  0001 C CNN
+F 2 "Capacitor_SMD:C_0805_2012Metric" H 7088 3125 50  0001 C CNN
 F 3 "~" H 7050 3275 50  0001 C CNN
 	1    7050 3275
@@
 P 7050 2975
 AR Path="/5CC6666B" Ref="C?"  Part="1"
-AR Path="/5CCFEC3E/5CC6666B" Ref="C5"  Part="1"
-F 0 "C5" V 6798 2975 50  0000 C CNN
+AR Path="/5CCFEC3E/5CC6666B" Ref="C4"  Part="1"
+F 0 "C4" V 6798 2975 50  0000 C CNN
 F 1 "22pF" V 6889 2975 50  0000 C CNN
-F 2 "Capacitor_SMD:C_0201_0603Metric" H 7088 2825 50  0001 C CNN
+F 2 "Capacitor_SMD:C_0805_2012Metric" H 7088 2825 50  0001 C CNN
 F 3 "~" H 7050 2975 50  0001 C CNN
 	1    7050 2975
@@
 LATCH_ADDR
 Text HLabel 5875 3525 2    50   Output ~ 0
-DATA_LED
+LATCH_LED
 $Comp
 L ftdi:FTDI J9
@@
 F 0 "R9" H 6770 3721 50  0000 L CNN
 F 1 "10K" H 6770 3630 50  0000 L CNN
-F 2 "Capacitor_SMD:C_0201_0603Metric" V 6630 3675 50  0001 C CNN
+F 2 "Resistor_SMD:R_0805_2012Metric" V 6630 3675 50  0001 C CNN
 F 3 "~" H 6700 3675 50  0001 C CNN
 	1    6700 3675
@@
 	7650 4025 8000 4025
 $Comp
-L Device:C C4
+L Device:C C3
 U 1 1 5CCED101
 P 6825 4200
-F 0 "C4" H 7025 4250 50  0000 L CNN
+F 0 "C3" H 7025 4250 50  0000 L CNN
 F 1 "100nF" H 6975 4150 50  0000 L CNN
-F 2 "Capacitor_SMD:C_0201_0603Metric" H 6863 4050 50  0001 C CNN
+F 2 "Capacitor_SMD:C_0805_2012Metric" H 6863 4050 50  0001 C CNN
 F 3 "~" H 6825 4200 50  0001 C CNN
 	1    6825 4200
@@
 F 0 "R10" H 8070 4371 50  0000 L CNN
 F 1 "4K7" H 8070 4280 50  0000 L CNN
-F 2 "Capacitor_SMD:C_0201_0603Metric" V 7930 4325 50  0001 C CNN
+F 2 "Resistor_SMD:R_0805_2012Metric" V 7930 4325 50  0001 C CNN
 F 3 "~" H 8000 4325 50  0001 C CNN
 	1    8000 4325
@@
 F 0 "R7" H 6275 4850 50  0000 L CNN
 F 1 "100R" V 6425 4600 50  0000 L CNN
-F 2 "Capacitor_SMD:C_0201_0603Metric" V 6355 4700 50  0001 C CNN
+F 2 "Resistor_SMD:R_0805_2012Metric" V 6355 4700 50  0001 C CNN
 F 3 "~" H 6425 4700 50  0001 C CNN
 	1    6425 4700
@@
 F 0 "R8" H 6425 4850 50  0000 L CNN
 F 1 "100R" V 6525 4600 50  0000 L CNN
-F 2 "Capacitor_SMD:C_0201_0603Metric" V 6455 4700 50  0001 C CNN
+F 2 "Resistor_SMD:R_0805_2012Metric" V 6455 4700 50  0001 C CNN
 F 3 "~" H 6525 4700 50  0001 C CNN
 	1    6525 4700
@@
 L Device:C C?
 U 1 1 5D1392AB
-P 3025 2700
+P 10050 2150
 AR Path="/5D1392AB" Ref="C?"  Part="1"
-AR Path="/5CCFEC3E/5D1392AB" Ref="C3"  Part="1"
-F 0 "C3" H 2800 2900 50  0000 L CNN
-F 1 "100nF" H 2750 2800 50  0000 L CNN
-F 2 "Capacitor_SMD:C_0201_0603Metric" H 3063 2550 50  0001 C CNN
-F 3 "~" H 3025 2700 50  0001 C CNN
-	1    3025 2700
-	1    0    0    -1
-$EndComp
-$Comp
-L power:VCC #PWR017
+AR Path="/5CCFEC3E/5D1392AB" Ref="C6"  Part="1"
+F 0 "C6" H 9825 2350 50  0000 L CNN
+F 1 "100nF" H 9775 2250 50  0000 L CNN
+F 2 "Capacitor_SMD:C_0805_2012Metric" H 10088 2000 50  0001 C CNN
+F 3 "~" H 10050 2150 50  0001 C CNN
+	1    10050 2150
+	1    0    0    -1
+$EndComp
+$Comp
+L power:VCC #PWR030
 U 1 1 5D13AC7F
-P 3025 2425
-F 0 "#PWR017" H 3025 2275 50  0001 C CNN
-F 1 "VCC" H 3042 2598 50  0000 C CNN
-F 2 "" H 3025 2425 50  0001 C CNN
-F 3 "" H 3025 2425 50  0001 C CNN
-	1    3025 2425
-	1    0    0    -1
-$EndComp
-$Comp
-L power:GND #PWR018
+P 10050 1775
+F 0 "#PWR030" H 10050 1625 50  0001 C CNN
+F 1 "VCC" H 10067 1948 50  0000 C CNN
+F 2 "" H 10050 1775 50  0001 C CNN
+F 3 "" H 10050 1775 50  0001 C CNN
+	1    10050 1775
+	1    0    0    -1
+$EndComp
+$Comp
+L power:GND #PWR031
 U 1 1 5D13B83C
-P 3025 2950
-F 0 "#PWR018" H 3025 2700 50  0001 C CNN
-F 1 "GND" H 3030 2777 50  0000 C CNN
-F 2 "" H 3025 2950 50  0001 C CNN
-F 3 "" H 3025 2950 50  0001 C CNN
-	1    3025 2950
-	1    0    0    -1
-$EndComp
-Wire Wire Line
-	3025 2425 3025 2550
-Wire Wire Line
-	3025 2850 3025 2950
-Text Notes 2650 2375 0    50   ~ 0
+P 10050 2400
+F 0 "#PWR031" H 10050 2150 50  0001 C CNN
+F 1 "GND" H 10055 2227 50  0000 C CNN
+F 2 "" H 10050 2400 50  0001 C CNN
+F 3 "" H 10050 2400 50  0001 C CNN
+	1    10050 2400
+	1    0    0    -1
+$EndComp
+Wire Wire Line
+	10050 2300 10050 2400
+Text Notes 9675 1725 0    50   ~ 0
 Bypass
 Wire Wire Line
@@
 F 0 "R13" V 8275 2575 50  0000 C CNN
 F 1 "4K7" V 8250 2750 50  0000 C CNN
-F 2 "Capacitor_SMD:C_0201_0603Metric" V 8180 2750 50  0001 C CNN
+F 2 "Resistor_SMD:R_0805_2012Metric" V 8180 2750 50  0001 C CNN
 F 3 "~" H 8250 2750 50  0001 C CNN
 	1    8250 2750
@@
 F 0 "R12" V 8175 2575 50  0000 C CNN
 F 1 "4K7" V 8150 2750 50  0000 C CNN
-F 2 "Capacitor_SMD:C_0201_0603Metric" V 8080 2750 50  0001 C CNN
+F 2 "Resistor_SMD:R_0805_2012Metric" V 8080 2750 50  0001 C CNN
 F 3 "~" H 8150 2750 50  0001 C CNN
 	1    8150 2750
@@
 F 0 "R11" V 8075 2575 50  0000 C CNN
 F 1 "4K7" V 8050 2750 50  0000 C CNN
-F 2 "Capacitor_SMD:C_0201_0603Metric" V 7980 2750 50  0001 C CNN
+F 2 "Resistor_SMD:R_0805_2012Metric" V 7980 2750 50  0001 C CNN
 F 3 "~" H 8050 2750 50  0001 C CNN
 	1    8050 2750
@@
 Wire Wire Line
 	6525 4450 6525 4550
-NoConn ~ 5875 2775
 Wire Wire Line
 	8250 2900 8150 2900
@@
 Wire Wire Line
 	8575 3750 8575 4050
+Text HLabel 5875 2775 2    50   Output ~ 0
+MOSI
+$Comp
+L Device:C C?
+U 1 1 5CD38628
+P 10375 2150
+AR Path="/5CD38628" Ref="C?"  Part="1"
+AR Path="/5CCFEC3E/5CD38628" Ref="C7"  Part="1"
+F 0 "C7" H 10150 2350 50  0000 L CNN
+F 1 "100nF" H 10100 2250 50  0000 L CNN
+F 2 "Capacitor_SMD:C_0805_2012Metric" H 10413 2000 50  0001 C CNN
+F 3 "~" H 10375 2150 50  0001 C CNN
+	1    10375 2150
+	1    0    0    -1
+$EndComp
+$Comp
+L power:GND #PWR032
+U 1 1 5CD3862E
+P 10375 2400
+F 0 "#PWR032" H 10375 2150 50  0001 C CNN
+F 1 "GND" H 10380 2227 50  0000 C CNN
+F 2 "" H 10375 2400 50  0001 C CNN
+F 3 "" H 10375 2400 50  0001 C CNN
+	1    10375 2400
+	1    0    0    -1
+$EndComp
+Wire Wire Line
+	10375 2300 10375 2400
+Wire Wire Line
+	10050 1775 10050 1900
+Wire Wire Line
+	10050 1900 10375 1900
+Wire Wire Line
+	10375 1900 10375 2000
+Wire Wire Line
+	10050 2000 10050 1900
+Connection ~ 10050 1900
 $EndSCHEMATC

Commit message: pcb: add testpads for SPI
Parts:
- added TP1: MISO, TestPoint:TestPoint_Pad_D1.0mm, symbol Connector:TestPoint
- added TP2: MOSI, TestPoint:TestPoint_Pad_D1.0mm, symbol Connector:TestPoint
- added TP3: SCK, TestPoint:TestPoint_Pad_D1.0mm, symbol Connector:TestPoint
- added TP4: RESET, TestPoint:TestPoint_Pad_D1.0mm, symbol Connector:TestPoint
- added TP5: VCC, TestPoint:TestPoint_Pad_D1.0mm, symbol Connector:TestPoint
- added TP6: GND, TestPoint:TestPoint_Pad_D1.0mm, symbol Connector:TestPoint
Connections:
- net GND: now also TP6.1
- net MISO: now also TP1.1
- net MOSI: now also TP2.1
- net SCK: now also TP3.1
- net VCC: now also TP5.1
- net RESET: now reaches C3.1, R9.2, SW2.1, U2.29 ((PCINT14/~RESET~)PC6)
- net RESET: now also TP4.1
Changed lines of the file:
@@
 Connection ~ 3625 4775
 Wire Wire Line
-	5825 3925 6700 3925
+	5825 3925 6500 3925
 Wire Wire Line
 	6825 3925 7250 3925
@@
 	10050 2000 10050 1900
 Connection ~ 10050 1900
+$Comp
+L Connector:TestPoint TP1
+U 1 1 5CD22E49
+P 8975 4675
+F 0 "TP1" V 8929 4863 50  0000 L CNN
+F 1 "MISO" V 9020 4863 50  0000 L CNN
+F 2 "TestPoint:TestPoint_Pad_D1.0mm" H 9175 4675 50  0001 C CNN
+F 3 "~" H 9175 4675 50  0001 C CNN
+	1    8975 4675
+	0    1    1    0
+$EndComp
+$Comp
+L Connector:TestPoint TP3
+U 1 1 5CD25980
+P 8975 5075
+F 0 "TP3" V 8929 5263 50  0000 L CNN
+F 1 "SCK" V 9020 5263 50  0000 L CNN
+F 2 "TestPoint:TestPoint_Pad_D1.0mm" H 9175 5075 50  0001 C CNN
+F 3 "~" H 9175 5075 50  0001 C CNN
+	1    8975 5075
+	0    1    1    0
+$EndComp
+$Comp
+L Connector:TestPoint TP5
+U 1 1 5CD25E18
+P 8975 5475
+F 0 "TP5" V 8929 5663 50  0000 L CNN
+F 1 "VCC" V 9020 5663 50  0000 L CNN
+F 2 "TestPoint:TestPoint_Pad_D1.0mm" H 9175 5475 50  0001 C CNN
+F 3 "~" H 9175 5475 50  0001 C CNN
+	1    8975 5475
+	0    1    1    0
+$EndComp
+$Comp
+L Connector:TestPoint TP2
+U 1 1 5CD2620B
+P 8975 4875
+F 0 "TP2" V 8929 5063 50  0000 L CNN
+F 1 "MOSI" V 9020 5063 50  0000 L CNN
+F 2 "TestPoint:TestPoint_Pad_D1.0mm" H 9175 4875 50  0001 C CNN
+F 3 "~" H 9175 4875 50  0001 C CNN
+	1    8975 4875
+	0    1    1    0
+$EndComp
+$Comp
+L Connector:TestPoint TP4
+U 1 1 5CD26549
+P 8975 5275
+F 0 "TP4" V 8929 5463 50  0000 L CNN
+F 1 "RESET" V 9020 5463 50  0000 L CNN
+F 2 "TestPoint:TestPoint_Pad_D1.0mm" H 9175 5275 50  0001 C CNN
+F 3 "~" H 9175 5275 50  0001 C CNN
+	1    8975 5275
+	0    1    1    0
+$EndComp
+$Comp
+L Connector:TestPoint TP6
+U 1 1 5CD26781
+P 8975 5675
+F 0 "TP6" V 8929 5863 50  0000 L CNN
+F 1 "GND" V 9020 5863 50  0000 L CNN
+F 2 "TestPoint:TestPoint_Pad_D1.0mm" H 9175 5675 50  0001 C CNN
+F 3 "~" H 9175 5675 50  0001 C CNN
+	1    8975 5675
+	0    1    1    0
+$EndComp
+Wire Wire Line
+	8975 4675 8875 4675
+Wire Wire Line
+	8975 4875 8875 4875
+Wire Wire Line
+	8975 5075 8875 5075
+Wire Wire Line
+	8975 5275 8875 5275
+Text HLabel 8875 4675 0    50   Input ~ 0
+MISO
+Text HLabel 8875 4875 0    50   Input ~ 0
+MOSI
+Text HLabel 8875 5075 0    50   Input ~ 0
+SCK
+Text Label 6500 3825 1    50   ~ 0
+RESET
+Wire Wire Line
+	6500 3825 6500 3925
+Connection ~ 6500 3925
+Wire Wire Line
+	6500 3925 6700 3925
+Text Label 8875 5275 2    50   ~ 0
+RESET
+$Comp
+L power:VCC #PWR0101
+U 1 1 5CD9E006
+P 8525 5475
+F 0 "#PWR0101" H 8525 5325 50  0001 C CNN
+F 1 "VCC" H 8542 5648 50  0000 C CNN
+F 2 "" H 8525 5475 50  0001 C CNN
+F 3 "" H 8525 5475 50  0001 C CNN
+	1    8525 5475
+	1    0    0    -1
+$EndComp
+$Comp
+L power:GND #PWR0102
+U 1 1 5CDA0796
+P 8525 5675
+F 0 "#PWR0102" H 8525 5425 50  0001 C CNN
+F 1 "GND" H 8530 5502 50  0000 C CNN
+F 2 "" H 8525 5675 50  0001 C CNN
+F 3 "" H 8525 5675 50  0001 C CNN
+	1    8525 5675
+	1    0    0    -1
+$EndComp
+Wire Wire Line
+	8525 5475 8975 5475
+Wire Wire Line
+	8525 5675 8975 5675
 $EndSCHEMATC

Commit message: pcb: add testpads for I2C
Parts:
- added TP7: SDA, TestPoint:TestPoint_Pad_D1.0mm, symbol Connector:TestPoint
- added TP8: SDL, TestPoint:TestPoint_Pad_D1.0mm, symbol Connector:TestPoint
Connections:
- net SCL: now also TP8.1
- net SDA: now also TP7.1
Changed lines of the file:
@@
 Wire Wire Line
 	8525 5675 8975 5675
+$Comp
+L Connector:TestPoint TP7
+U 1 1 5CD64B91
+P 10300 3400
+F 0 "TP7" V 10254 3588 50  0000 L CNN
+F 1 "SDA" V 10345 3588 50  0000 L CNN
+F 2 "TestPoint:TestPoint_Pad_D1.0mm" H 10500 3400 50  0001 C CNN
+F 3 "~" H 10500 3400 50  0001 C CNN
+	1    10300 3400
+	0    1    1    0
+$EndComp
+$Comp
+L Connector:TestPoint TP8
+U 1 1 5CD65B22
+P 10300 3625
+F 0 "TP8" V 10254 3813 50  0000 L CNN
+F 1 "SDL" V 10345 3813 50  0000 L CNN
+F 2 "TestPoint:TestPoint_Pad_D1.0mm" H 10500 3625 50  0001 C CNN
+F 3 "~" H 10500 3625 50  0001 C CNN
+	1    10300 3625
+	0    1    1    0
+$EndComp
+Text Label 10200 3400 2    50   ~ 0
+SDA
+Text Label 10200 3625 2    50   ~ 0
+SCL
+Wire Wire Line
+	10300 3400 10200 3400
+Wire Wire Line
+	10300 3625 10200 3625
 $EndSCHEMATC

Commit message: pcb: add missing footprints / add component for logo footprint
Parts:
- added T1: Logo, logo:logo, symbol ibm_pc_floppy_idc:Logo
Changed lines of the file:
@@
 Wire Wire Line
 	10300 3625 10200 3625
+$Comp
+L ibm_pc_floppy_idc:Logo T1
+U 1 1 5CE030CA
+P 6150 1725
+F 0 "T1" H 6175 1775 50  0001 C CNN
+F 1 "Logo" H 6328 1725 50  0000 L CNN
+F 2 "logo:logo" H 6150 1725 50  0001 C CNN
+F 3 "" H 6150 1725 50  0001 C CNN
+	1    6150 1725
+	1    0    0    -1
+$EndComp
 $EndSCHEMATC
