File: Arduino/pcb/mcu.sch (KiCad schematic (older format))
At the start: 27 parts, among them J9 FTDI, SW2 Reset Button, U2 ATMEGA328P-AU, U3 24LC64, U5 74AHC1G08, Y1 20 Mhz Crystal

Commit message: pcb: do some final optimizations for v3.1
Parts:
- added J10: AVR-ISP-6, Connector_PinHeader_2.54mm:PinHeader_2x03_P2.54mm_Vertical, symbol Connector:AVR-ISP-6
Connections:
- net 5V_ISP: now also TP5.1, J10.2 (VCC)
- net GND: now also J10.6 (GND)
- net MISO: now also J10.1 (MISO)
- net MOSI: now also J10.4 (MOSI)
- net RESET: now also J10.5 (~RST)
- net SCK: now also J10.3 (SCK)
- net VCC: no longer TP5.1
Other:
- moved on the sheet: TP1, TP2, TP3, TP4, TP5, TP6, TP7, TP8
Changed lines of the file:
@@
 L Connector:TestPoint TP1
 U 1 1 5CD22E49
-P 9125 4750
-F 0 "TP1" V 9079 4938 50  0000 L CNN
-F 1 "MISO" V 9170 4938 50  0000 L CNN
-F 2 "TestPoint:TestPoint_Pad_D1.0mm" H 9325 4750 50  0001 C CNN
-F 3 "~" H 9325 4750 50  0001 C CNN
-	1    9125 4750
+P 10000 5025
+F 0 "TP1" V 10000 5225 50  0000 L CNN
+F 1 "MISO" V 10000 5400 50  0000 L CNN
+F 2 "TestPoint:TestPoint_Pad_D1.0mm" H 10200 5025 50  0001 C CNN
+F 3 "~" H 10200 5025 50  0001 C CNN
+	1    10000 5025
 	0    1    1    0
 $EndComp
@@
 L Connector:TestPoint TP3
 U 1 1 5CD25980
-P 9125 5150
-F 0 "TP3" V 9079 5338 50  0000 L CNN
-F 1 "SCK" V 9170 5338 50  0000 L CNN
-F 2 "TestPoint:TestPoint_Pad_D1.0mm" H 9325 5150 50  0001 C CNN
-F 3 "~" H 9325 5150 50  0001 C CNN
-	1    9125 5150
+P 10000 5225
+F 0 "TP3" V 10000 5425 50  0000 L CNN
+F 1 "SCK" V 10000 5600 50  0000 L CNN
+F 2 "TestPoint:TestPoint_Pad_D1.0mm" H 10200 5225 50  0001 C CNN
+F 3 "~" H 10200 5225 50  0001 C CNN
+	1    10000 5225
 	0    1    1    0
 $EndComp
@@
 L Connector:TestPoint TP5
 U 1 1 5CD25E18
-P 9125 5550
-F 0 "TP5" V 9079 5738 50  0000 L CNN
-F 1 "VCC" V 9170 5738 50  0000 L CNN
-F 2 "TestPoint:TestPoint_Pad_D1.0mm" H 9325 5550 50  0001 C CNN
-F 3 "~" H 9325 5550 50  0001 C CNN
-	1    9125 5550
-	0    1    1    0
-$EndComp
-$Comp
-L Connector:TestPoint TP2
-U 1 1 5CD2620B
-P 9125 4950
-F 0 "TP2" V 9079 5138 50  0000 L CNN
-F 1 "MOSI" V 9170 5138 50  0000 L CNN
-F 2 "TestPoint:TestPoint_Pad_D1.0mm" H 9325 4950 50  0001 C CNN
-F 3 "~" H 9325 4950 50  0001 C CNN
-	1    9125 4950
-	0    1    1    0
-$EndComp
-$Comp
-L Connector:TestPoint TP4
-U 1 1 5CD26549
-P 9125 5350
-F 0 "TP4" V 9079 5538 50  0000 L CNN
-F 1 "RESET" V 9170 5538 50  0000 L CNN
-F 2 "TestPoint:TestPoint_Pad_D1.0mm" H 9325 5350 50  0001 C CNN
-F 3 "~" H 9325 5350 50  0001 C CNN
-	1    9125 5350
+P 9775 4700
+F 0 "TP5" V 9675 4775 50  0000 L CNN
+F 1 "VCC" V 9675 4950 50  0000 L CNN
+F 2 "TestPoint:TestPoint_Pad_D1.0mm" H 9975 4700 50  0001 C CNN
+F 3 "~" H 9975 4700 50  0001 C CNN
+	1    9775 4700
 	0    1    1    0
 $EndComp
@@
 L Connector:TestPoint TP6
 U 1 1 5CD26781
-P 9125 5750
-F 0 "TP6" V 9079 5938 50  0000 L CNN
-F 1 "GND" V 9170 5938 50  0000 L CNN
-F 2 "TestPoint:TestPoint_Pad_D1.0mm" H 9325 5750 50  0001 C CNN
-F 3 "~" H 9325 5750 50  0001 C CNN
-	1    9125 5750
+P 9775 5650
+F 0 "TP6" V 9675 5725 50  0000 L CNN
+F 1 "GND" V 9675 5900 50  0000 L CNN
+F 2 "TestPoint:TestPoint_Pad_D1.0mm" H 9975 5650 50  0001 C CNN
+F 3 "~" H 9975 5650 50  0001 C CNN
+	1    9775 5650
 	0    1    1    0
 $EndComp
 Wire Wire Line
-	9125 4750 9025 4750
-Wire Wire Line
-	9125 4950 9025 4950
-Wire Wire Line
-	9125 5150 9025 5150
-Wire Wire Line
-	9125 5350 9025 5350
-Wire Wire Line
 	6500 3825 6500 3925
 Connection ~ 6500 3925
 Wire Wire Line
 	6500 3925 6700 3925
-Text Label 9025 5350 2    50   ~ 0
-RESET
-$Comp
-L power:VCC #PWR026
-U 1 1 5CD9E006
-P 8675 5550
-F 0 "#PWR026" H 8675 5400 50  0001 C CNN
-F 1 "VCC" H 8692 5723 50  0000 C CNN
-F 2 "" H 8675 5550 50  0001 C CNN
-F 3 "" H 8675 5550 50  0001 C CNN
-	1    8675 5550
-	1    0    0    -1
-$EndComp
 $Comp
 L power:GND #PWR027
 U 1 1 5CDA0796
-P 8675 5750
-F 0 "#PWR027" H 8675 5500 50  0001 C CNN
-F 1 "GND" H 8680 5577 50  0000 C CNN
-F 2 "" H 8675 5750 50  0001 C CNN
-F 3 "" H 8675 5750 50  0001 C CNN
-	1    8675 5750
+P 9325 5700
+F 0 "#PWR027" H 9325 5450 50  0001 C CNN
+F 1 "GND" H 9330 5527 50  0000 C CNN
+F 2 "" H 9325 5700 50  0001 C CNN
+F 3 "" H 9325 5700 50  0001 C CNN
+	1    9325 5700
 	1    0    0    -1
 $EndComp
 Wire Wire Line
-	8675 5550 9125 5550
+	9325 4700 9775 4700
 Wire Wire Line
-	8675 5750 9125 5750
+	9325 5650 9775 5650
 $Comp
 L Connector:TestPoint TP7
 U 1 1 5CD64B91
-P 10225 5100
-F 0 "TP7" V 10179 5288 50  0000 L CNN
-F 1 "SDA" V 10270 5288 50  0000 L CNN
-F 2 "TestPoint:TestPoint_Pad_D1.0mm" H 10425 5100 50  0001 C CNN
-F 3 "~" H 10425 5100 50  0001 C CNN
-	1    10225 5100
+P 10775 3550
+F 0 "TP7" V 10729 3738 50  0000 L CNN
+F 1 "SDA" V 10820 3738 50  0000 L CNN
+F 2 "TestPoint:TestPoint_Pad_D1.0mm" H 10975 3550 50  0001 C CNN
+F 3 "~" H 10975 3550 50  0001 C CNN
+	1    10775 3550
 	0    1    1    0
 $EndComp
@@
 L Connector:TestPoint TP8
 U 1 1 5CD65B22
-P 10225 5325
-F 0 "TP8" V 10179 5513 50  0000 L CNN
-F 1 "SDL" V 10270 5513 50  0000 L CNN
-F 2 "TestPoint:TestPoint_Pad_D1.0mm" H 10425 5325 50  0001 C CNN
-F 3 "~" H 10425 5325 50  0001 C CNN
-	1    10225 5325
+P 10775 3775
+F 0 "TP8" V 10729 3963 50  0000 L CNN
+F 1 "SDL" V 10820 3963 50  0000 L CNN
+F 2 "TestPoint:TestPoint_Pad_D1.0mm" H 10975 3775 50  0001 C CNN
+F 3 "~" H 10975 3775 50  0001 C CNN
+	1    10775 3775
 	0    1    1    0
 $EndComp
-Text Label 10125 5100 2    50   ~ 0
+Text Label 10675 3550 2    50   ~ 0
 SDA
-Text Label 10125 5325 2    50   ~ 0
+Text Label 10675 3775 2    50   ~ 0
 SCL
 Wire Wire Line
-	10225 5100 10125 5100
+	10775 3550 10675 3550
 Wire Wire Line
-	10225 5325 10125 5325
+	10775 3775 10675 3775
 Text Label 6500 3825 1    50   ~ 0
 RESET
@@
 Text Label 5875 2975 0    50   ~ 0
 SCK
-Text Label 9025 4750 2    50   ~ 0
+Text Label 9900 5025 0    50   ~ 0
 MISO
-Text Label 9025 4950 2    50   ~ 0
-MOSI
-Text Label 9025 5150 2    50   ~ 0
+Text Label 9900 5225 0    50   ~ 0
 SCK
 Text Label 7975 2500 1    50   ~ 0
@@
 Wire Wire Line
 	3825 3925 3925 3925
+$Comp
+L Connector:AVR-ISP-6 J10
+U 1 1 5D9FFF31
+P 9425 5225
+F 0 "J10" H 9146 5321 50  0000 R CNN
+F 1 "AVR-ISP-6" H 9146 5230 50  0000 R CNN
+F 2 "Connector_PinHeader_2.54mm:PinHeader_2x03_P2.54mm_Vertical" V 9175 5275 50  0001 C CNN
+F 3 " ~" H 8150 4675 50  0001 C CNN
+	1    9425 5225
+	1    0    0    -1
+$EndComp
+Wire Wire Line
+	9325 5625 9325 5650
+Connection ~ 9325 5650
+Wire Wire Line
+	9325 5650 9325 5700
+Wire Wire Line
+	9325 4700 9325 4725
+$Comp
+L Connector:TestPoint TP4
+U 1 1 5CD26549
+P 10000 5325
+F 0 "TP4" V 10000 5525 50  0000 L CNN
+F 1 "RESET" V 10000 5700 50  0000 L CNN
+F 2 "TestPoint:TestPoint_Pad_D1.0mm" H 10200 5325 50  0001 C CNN
+F 3 "~" H 10200 5325 50  0001 C CNN
+	1    10000 5325
+	0    1    1    0
+$EndComp
+Text Label 9900 5325 0    50   ~ 0
+RESET
+Wire Wire Line
+	9825 5025 10000 5025
+Text Label 9900 5125 0    50   ~ 0
+MOSI
+$Comp
+L Connector:TestPoint TP2
+U 1 1 5CD2620B
+P 10000 5125
+F 0 "TP2" V 10000 5325 50  0000 L CNN
+F 1 "MOSI" V 10000 5500 50  0000 L CNN
+F 2 "TestPoint:TestPoint_Pad_D1.0mm" H 10200 5125 50  0001 C CNN
+F 3 "~" H 10200 5125 50  0001 C CNN
+	1    10000 5125
+	0    1    1    0
+$EndComp
+Wire Wire Line
+	9825 5125 10000 5125
+Wire Wire Line
+	9825 5225 10000 5225
+Wire Wire Line
+	9825 5325 10000 5325
+Text HLabel 9225 4600 0    50   Output ~ 0
+5V_ISP
+Wire Wire Line
+	9325 4700 9325 4600
+Wire Wire Line
+	9325 4600 9225 4600
+Connection ~ 9325 4700
 $EndSCHEMATC

Commit message: migrate to kicad 5.x
Parts:
- J10: symbol Connector:AVR-ISP-6 -> floppyorgel-rescue:AVR-ISP-6-Connector
Changed lines of the file:
@@
 EESchema Schematic File Version 4
-LIBS:floppyorgel-cache
 EELAYER 30 0
 EELAYER END
@@
 	3825 3925 3925 3925
 $Comp
-L Connector:AVR-ISP-6 J10
+L floppyorgel-rescue:AVR-ISP-6-Connector J10
 U 1 1 5D9FFF31
 P 9425 5225
+AR Path="/5D9FFF31" Ref="J10"  Part="1"
+AR Path="/5CCFEC3E/5D9FFF31" Ref="J10"  Part="1"
 F 0 "J10" H 9146 5321 50  0000 R CNN
 F 1 "AVR-ISP-6" H 9146 5230 50  0000 R CNN

Commit message: pcb: reannotate symbols
Parts:
- renumbered C5 to C1, C4 to C2, C6 to C4, C7 to C5, J9 to J4, J10 to J5, R12 to R10, R13 to R11, R10 to R12, R20 to R13, R21 to R14, R9 to R7, R7 to R8, R8 to R9, SW2 to SW1, TP5 to TP1, TP6 to TP2, TP1 to TP3, TP2 to TP4, TP3 to TP5, TP4 to TP6, U2 to U1, U5 to U2
Connections:
- net at U1.8 ((PCINT7/XTAL2/TOSC2)PB7), Y1.1: now also C2.2; no longer C1.1
- net at U1.7 ((PCINT6/XTAL1/TOSC1)PB6), Y1.2: now also C1.1; no longer C2.2
Other:
- moved on the sheet: C1, C2
