File: Arduino/pcb/led.sch (KiCad schematic (older format))
At the start: 12 parts, among them Q1 IRLML2060, Q2 IRLML2060, Q3 IRLML2060, U4 74HC595

Commit message: pcb: add footprint for RGB led
Parts:
- D1: footprint LED_SMD:LED_RGB_1210 -> rgb_led:rgb_led_0805_2012Metric
Changed lines of the file:
@@
 F 0 "D1" H 6625 2622 50  0000 C CNN
 F 1 "LED_RGB" H 6625 2531 50  0000 C CNN
-F 2 "LED_SMD:LED_RGB_1210" H 6625 2075 50  0001 C CNN
+F 2 "rgb_led:rgb_led_0805_2012Metric" H 6625 2075 50  0001 C CNN
 F 3 "~" H 6625 2075 50  0001 C CNN
 	1    6625 2125

Commit message: pcb: fix rgb led footprint
Parts:
- removed D1: LED_RGB, rgb_led:rgb_led_0805_2012Metric, symbol Device:LED_RGB
- added D1: CHANZON_ARGB_LED, rgb_led:rgb_led_0805_2012Metric, symbol rgb_led:CHANZON_ARGB_LED
- renumbered R17 to R14, R18 to R15, R19 to R16, R14 to R17, R15 to R18, R16 to R19
Connections:
- net VCC: now also D1.3 (COM); no longer R17.2, R18.2, R19.2
- net at R18.1: now also Q2.3 (D)
- net at R17.1: now also Q3.3 (D)
- net at R19.1: now also Q1.3 (D)
- new net: D1.2 (GK), R18.2
- new net: D1.1 (RK), R17.2
- new net: D1.4 (BK), R19.2
Other:
- moved on the sheet: Q1, Q2, Q3, R17, R18, R19
Changed lines of the file:
@@
 Bypass
 $Comp
-L Device:R R15
+L Device:R R18
 U 1 1 5CDFA92E
-P 6075 2125
-F 0 "R15" V 6025 1925 50  0000 C CNN
-F 1 "250R" V 6075 2125 50  0000 C CNN
-F 2 "Resistor_SMD:R_0805_2012Metric" V 6005 2125 50  0001 C CNN
-F 3 "~" H 6075 2125 50  0001 C CNN
-	1    6075 2125
+P 6925 2125
+F 0 "R18" V 6875 1925 50  0000 C CNN
+F 1 "250R" V 6925 2125 50  0000 C CNN
+F 2 "Resistor_SMD:R_0805_2012Metric" V 6855 2125 50  0001 C CNN
+F 3 "~" H 6925 2125 50  0001 C CNN
+	1    6925 2125
 	0    1    1    0
 $EndComp
 $Comp
-L Device:R R14
+L Device:R R17
 U 1 1 5CDFACA1
-P 6075 2025
-F 0 "R14" V 6025 1825 50  0000 C CNN
-F 1 "250R" V 6075 2025 50  0000 C CNN
-F 2 "Resistor_SMD:R_0805_2012Metric" V 6005 2025 50  0001 C CNN
-F 3 "~" H 6075 2025 50  0001 C CNN
-	1    6075 2025
+P 6925 1925
+F 0 "R17" V 6875 1725 50  0000 C CNN
+F 1 "250R" V 6925 1925 50  0000 C CNN
+F 2 "Resistor_SMD:R_0805_2012Metric" V 6855 1925 50  0001 C CNN
+F 3 "~" H 6925 1925 50  0001 C CNN
+	1    6925 1925
 	0    1    1    0
 $EndComp
@@
 L power:GND #PWR043
 U 1 1 5CE5B10B
-P 6975 3150
-F 0 "#PWR043" H 6975 2900 50  0001 C CNN
-F 1 "GND" H 6980 2977 50  0000 C CNN
-F 2 "" H 6975 3150 50  0001 C CNN
-F 3 "" H 6975 3150 50  0001 C CNN
-	1    6975 3150
+P 7250 3150
+F 0 "#PWR043" H 7250 2900 50  0001 C CNN
+F 1 "GND" H 7255 2977 50  0000 C CNN
+F 2 "" H 7250 3150 50  0001 C CNN
+F 3 "" H 7250 3150 50  0001 C CNN
+	1    7250 3150
 	1    0    0    -1
 $EndComp
@@
 L Transistor_FET:IRLML2060 Q1
 U 1 1 5CE57929
-P 6875 2950
-F 0 "Q1" H 7100 2975 50  0000 L CNN
-F 1 "IRLML2060" H 7100 2900 50  0000 L CNN
-F 2 "Package_TO_SOT_SMD:SOT-23" H 7075 2875 50  0001 L CIN
-F 3 "https://www.infineon.com/dgdl/irlml2060pbf.pdf?fileId=5546d462533600a401535664b7fb25ee" H 6875 2950 50  0001 L CNN
-	1    6875 2950
-	1    0    0    -1
-$EndComp
-Wire Wire Line
-	6225 2225 6225 2325
-Wire Wire Line
-	6225 2025 6225 1925
-$Comp
-L Device:LED_RGB D1
-U 1 1 5D09B2AA
-P 6625 2125
-F 0 "D1" H 6625 2622 50  0000 C CNN
-F 1 "LED_RGB" H 6625 2531 50  0000 C CNN
-F 2 "rgb_led:rgb_led_0805_2012Metric" H 6625 2075 50  0001 C CNN
-F 3 "~" H 6625 2075 50  0001 C CNN
-	1    6625 2125
-	-1   0    0    -1
-$EndComp
-$Comp
-L Device:R R16
+P 7150 2950
+F 0 "Q1" H 7375 2975 50  0000 L CNN
+F 1 "IRLML2060" H 7375 2900 50  0000 L CNN
+F 2 "Package_TO_SOT_SMD:SOT-23" H 7350 2875 50  0001 L CIN
+F 3 "https://www.infineon.com/dgdl/irlml2060pbf.pdf?fileId=5546d462533600a401535664b7fb25ee" H 7150 2950 50  0001 L CNN
+	1    7150 2950
+	1    0    0    -1
+$EndComp
+$Comp
+L Device:R R19
 U 1 1 5CDFAF66
-P 6075 2225
-F 0 "R16" V 6025 2025 50  0000 C CNN
-F 1 "170R" V 6075 2225 50  0000 C CNN
-F 2 "Resistor_SMD:R_0805_2012Metric" V 6005 2225 50  0001 C CNN
-F 3 "~" H 6075 2225 50  0001 C CNN
-	1    6075 2225
+P 6925 2325
+F 0 "R19" V 6875 2125 50  0000 C CNN
+F 1 "170R" V 6925 2325 50  0000 C CNN
+F 2 "Resistor_SMD:R_0805_2012Metric" V 6855 2325 50  0001 C CNN
+F 3 "~" H 6925 2325 50  0001 C CNN
+	1    6925 2325
 	0    1    1    0
 $EndComp
@@
 L power:VCC #PWR041
 U 1 1 5CEB296C
-P 5725 1925
-F 0 "#PWR041" H 5725 1775 50  0001 C CNN
-F 1 "VCC" H 5742 2098 50  0000 C CNN
-F 2 "" H 5725 1925 50  0001 C CNN
-F 3 "" H 5725 1925 50  0001 C CNN
-	1    5725 1925
-	1    0    0    -1
-$EndComp
-Connection ~ 5725 2025
-Wire Wire Line
-	5725 2025 5725 1925
-Connection ~ 5725 2125
-Wire Wire Line
-	5725 2025 5725 2125
-Wire Wire Line
-	5725 2225 5725 2125
-Wire Wire Line
-	5725 2025 5925 2025
-Wire Wire Line
-	5725 2125 5925 2125
-Wire Wire Line
-	5725 2225 5925 2225
+P 5975 1725
+F 0 "#PWR041" H 5975 1575 50  0001 C CNN
+F 1 "VCC" H 5992 1898 50  0000 C CNN
+F 2 "" H 5975 1725 50  0001 C CNN
+F 3 "" H 5975 1725 50  0001 C CNN
+	1    5975 1725
+	1    0    0    -1
+$EndComp
 $Comp
 L Transistor_FET:IRLML2060 Q2
 U 1 1 5CEEBDE6
-P 7125 3425
-F 0 "Q2" H 7331 3471 50  0000 L CNN
-F 1 "IRLML2060" H 7331 3380 50  0000 L CNN
-F 2 "Package_TO_SOT_SMD:SOT-23" H 7325 3350 50  0001 L CIN
-F 3 "https://www.infineon.com/dgdl/irlml2060pbf.pdf?fileId=5546d462533600a401535664b7fb25ee" H 7125 3425 50  0001 L CNN
-	1    7125 3425
-	1    0    0    -1
-$EndComp
-Wire Wire Line
-	6825 2125 7225 2125
+P 7400 3425
+F 0 "Q2" H 7606 3471 50  0000 L CNN
+F 1 "IRLML2060" H 7606 3380 50  0000 L CNN
+F 2 "Package_TO_SOT_SMD:SOT-23" H 7600 3350 50  0001 L CIN
+F 3 "https://www.infineon.com/dgdl/irlml2060pbf.pdf?fileId=5546d462533600a401535664b7fb25ee" H 7400 3425 50  0001 L CNN
+	1    7400 3425
+	1    0    0    -1
+$EndComp
 $Comp
 L power:GND #PWR044
 U 1 1 5CF166DE
-P 7225 3625
-F 0 "#PWR044" H 7225 3375 50  0001 C CNN
-F 1 "GND" H 7230 3452 50  0000 C CNN
-F 2 "" H 7225 3625 50  0001 C CNN
-F 3 "" H 7225 3625 50  0001 C CNN
-	1    7225 3625
+P 7500 3625
+F 0 "#PWR044" H 7500 3375 50  0001 C CNN
+F 1 "GND" H 7505 3452 50  0000 C CNN
+F 2 "" H 7500 3625 50  0001 C CNN
+F 3 "" H 7500 3625 50  0001 C CNN
+	1    7500 3625
 	1    0    0    -1
 $EndComp
@@
 L Transistor_FET:IRLML2060 Q3
 U 1 1 5CF1AF82
-P 7400 3900
-F 0 "Q3" H 7606 3946 50  0000 L CNN
-F 1 "IRLML2060" H 7606 3855 50  0000 L CNN
-F 2 "Package_TO_SOT_SMD:SOT-23" H 7600 3825 50  0001 L CIN
-F 3 "https://www.infineon.com/dgdl/irlml2060pbf.pdf?fileId=5546d462533600a401535664b7fb25ee" H 7400 3900 50  0001 L CNN
-	1    7400 3900
+P 7675 3900
+F 0 "Q3" H 7881 3946 50  0000 L CNN
+F 1 "IRLML2060" H 7881 3855 50  0000 L CNN
+F 2 "Package_TO_SOT_SMD:SOT-23" H 7875 3825 50  0001 L CIN
+F 3 "https://www.infineon.com/dgdl/irlml2060pbf.pdf?fileId=5546d462533600a401535664b7fb25ee" H 7675 3900 50  0001 L CNN
+	1    7675 3900
 	1    0    0    -1
 $EndComp
@@
 L power:GND #PWR045
 U 1 1 5CF1E097
-P 7500 4100
-F 0 "#PWR045" H 7500 3850 50  0001 C CNN
-F 1 "GND" H 7505 3927 50  0000 C CNN
-F 2 "" H 7500 4100 50  0001 C CNN
-F 3 "" H 7500 4100 50  0001 C CNN
-	1    7500 4100
-	1    0    0    -1
-$EndComp
-Wire Wire Line
-	6825 2325 6975 2325
-Wire Wire Line
-	6975 2325 6975 2750
-Wire Wire Line
-	7225 3225 7225 2125
-Wire Wire Line
-	7500 1925 7500 3700
-Wire Wire Line
-	6825 1925 7500 1925
+P 7775 4100
+F 0 "#PWR045" H 7775 3850 50  0001 C CNN
+F 1 "GND" H 7780 3927 50  0000 C CNN
+F 2 "" H 7775 4100 50  0001 C CNN
+F 3 "" H 7775 4100 50  0001 C CNN
+	1    7775 4100
+	1    0    0    -1
+$EndComp
+Wire Wire Line
+	7500 3225 7500 2125
+Wire Wire Line
+	7775 1925 7775 3700
 Wire Wire Line
 	6175 2950 6300 2950
-Wire Wire Line
-	6225 1925 6425 1925
-Wire Wire Line
-	6225 2125 6425 2125
-Wire Wire Line
-	6225 2325 6425 2325
-$Comp
-L Device:R R17
+$Comp
+L Device:R R14
 U 1 1 5CF4F3BC
 P 6300 4250
-F 0 "R17" V 6250 4375 50  0000 L CNN
+F 0 "R14" V 6250 4375 50  0000 L CNN
 F 1 "4k7" V 6300 4175 50  0000 L CNN
 F 2 "Resistor_SMD:R_0805_2012Metric" V 6230 4250 50  0001 C CNN
@@
 $EndComp
 $Comp
-L Device:R R18
+L Device:R R15
 U 1 1 5CF563D6
 P 6400 4250
-F 0 "R18" V 6350 4375 50  0000 L CNN
+F 0 "R15" V 6350 4375 50  0000 L CNN
 F 1 "4k7" V 6400 4175 50  0000 L CNN
 F 2 "Resistor_SMD:R_0805_2012Metric" V 6330 4250 50  0001 C CNN
@@
 $EndComp
 $Comp
-L Device:R R19
+L Device:R R16
 U 1 1 5CF56A72
 P 6500 4250
-F 0 "R19" V 6450 4375 50  0000 L CNN
+F 0 "R16" V 6450 4375 50  0000 L CNN
 F 1 "4k7" V 6500 4175 50  0000 L CNN
 F 2 "Resistor_SMD:R_0805_2012Metric" V 6430 4250 50  0001 C CNN
@@
 $EndComp
 Connection ~ 6300 2950
-Wire Wire Line
-	6300 2950 6675 2950
 $Comp
 L power:GND #PWR042
@@
 	6500 3150 6650 3150
 Wire Wire Line
-	6925 3425 6750 3425
-Wire Wire Line
 	6650 3150 6650 3900
-Wire Wire Line
-	6650 3900 7200 3900
 Wire Wire Line
 	6300 4400 6400 4400
@@
 Wire Wire Line
 	6500 3150 6500 4100
+Wire Wire Line
+	6650 3900 7475 3900
+Wire Wire Line
+	6750 3425 7200 3425
+Wire Wire Line
+	6300 2950 6950 2950
+Wire Wire Line
+	7250 2750 7250 2325
+Wire Wire Line
+	5975 2125 6200 2125
+Wire Wire Line
+	6600 1925 6775 1925
+Wire Wire Line
+	7075 1925 7775 1925
+Wire Wire Line
+	7075 2125 7500 2125
+Wire Wire Line
+	7075 2325 7250 2325
+Wire Wire Line
+	6600 2125 6775 2125
+Wire Wire Line
+	6600 2325 6775 2325
+$Comp
+L rgb_led:CHANZON_ARGB_LED D1
+U 1 1 5D002E41
+P 6400 2125
+F 0 "D1" H 6400 1658 50  0000 C CNN
+F 1 "CHANZON_ARGB_LED" H 6400 1749 50  0000 C CNN
+F 2 "rgb_led:rgb_led_0805_2012Metric" H 6400 2075 50  0001 C CNN
+F 3 "~" H 6400 2075 50  0001 C CNN
+	1    6400 2125
+	-1   0    0    -1
+$EndComp
+Wire Wire Line
+	5975 1725 5975 2125
 $EndSCHEMATC
