File: Arduino/pcb/floppy.sch (KiCad schematic (older format))
At the start: 0 parts

Commit message: pcb: continue wiring / move parts to hierachival sheets
Parts:
- added J2: Floppy-Power, floppy_power:Floppy_Power_1x04_Pitch2.54mm, symbol floppy-power:Floppy-Power
- added J3: IBM_PC_Floppy_IDC, Connector_PinHeader_2.54mm:PinHeader_2x17_P2.54mm_Horizontal, symbol ibm_pc_floppy_idc:IBM_PC_Floppy_IDC
- added R1, R2, R3, R4, R5, R6: 4K7, symbol Device:R
- added SW1: Bus Address Select, Buttons_Switches_THT:SW_DIP_x6_W7.62mm_Slide, symbol floppyorgel-rescue:SW_DIP_x06-switches
- added U1: 4021, symbol 4xxx_IEEE:4021
Connections:
- new net: R4.1, SW1.10, U1.5 (P2)
- new net: R5.1, SW1.11, U1.6 (P1)
- new net: R6.1, SW1.12, U1.7 (P0)
- new net: R1.1, SW1.7, U1.14 (P5)
- new net: R2.1, SW1.8, U1.13 (P4)
- new net: R3.1, SW1.9, U1.4 (P3)
- new net 12V_BUS: J2.4 (12V)
- new net 5V_BUS: J2.1 (5V)
- new net DIRECTION: J3.18 (Pin_18)
- new net DRIVE_SELECT: J3.12 (Pin_12)
- new net GND: J2.2 (Ground), J2.3 (Ground), J3.1 (Pin_1), J3.11 (Pin_11), J3.13 (Pin_13), J3.15 (Pin_15), J3.17 (Pin_17), J3.19 (Pin_19), J3.21 (Pin_21), J3.23 (Pin_23), J3.25 (Pin_25), J3.27 (Pin_27), J3.29 (Pin_29), J3.3 (Pin_3), J3.31 (Pin_31), J3.33 (Pin_33), J3.5 (Pin_5), J3.7 (Pin_7), J3.9 (Pin_9), R1.2, R2.2, R3.2, R4.2, R5.2, R6.2, U1.1 (P7), U1.11 (DS), U1.15 (P6), U1.8 (Vss)
- new net LATCH_ADDR: U1.9 (PL)
- new net MISO: U1.3 (Q7)
- new net SCK: U1.10 (CP)
- new net STEP: J3.20 (Pin_20)
- new net TRK00: J3.26 (Pin_26)
- new net VCC: SW1.1, SW1.2, SW1.3, SW1.4, SW1.5, SW1.6, U1.16 (Vdd)
- no-connect marks 0 -> 13

Commit message: pcb: finish wiring / use ws2812 under chip led
Parts:
- renumbered J2 to J7, J3 to J8
Changed lines of the file:
@@
 $Descr A4 11693 8268
 encoding utf-8
-Sheet 2 6
+Sheet 5 6
 Title ""
 Date ""
@@
 P 6875 3425
 AR Path="/5CE26438" Ref="J?"  Part="1"
-AR Path="/5CD0EE48/5CE26438" Ref="J3"  Part="1"
-F 0 "J3" H 7075 4475 50  0000 C CNN
+AR Path="/5CD0EE48/5CE26438" Ref="J8"  Part="1"
+F 0 "J8" H 7075 4475 50  0000 C CNN
 F 1 "IBM_PC_Floppy_IDC" H 7125 4375 50  0000 C CNN
 F 2 "Connector_PinHeader_2.54mm:PinHeader_2x17_P2.54mm_Horizontal" H 6875 3425 50  0001 C CNN
@@
 P 7075 4425
 AR Path="/5CE2645F" Ref="#PWR?"  Part="1"
-AR Path="/5CD0EE48/5CE2645F" Ref="#PWR08"  Part="1"
-F 0 "#PWR08" H 7075 4175 50  0001 C CNN
+AR Path="/5CD0EE48/5CE2645F" Ref="#PWR017"  Part="1"
+F 0 "#PWR017" H 7075 4175 50  0001 C CNN
 F 1 "GND" H 7080 4252 50  0000 C CNN
 F 2 "" H 7075 4425 50  0001 C CNN
@@
 P 1975 1925
 AR Path="/5CEBDDC6" Ref="J?"  Part="1"
-AR Path="/5CD0EE48/5CEBDDC6" Ref="J2"  Part="1"
-F 0 "J2" H 2025 2275 50  0000 L CNN
+AR Path="/5CD0EE48/5CEBDDC6" Ref="J7"  Part="1"
+F 0 "J7" H 2025 2275 50  0000 L CNN
 F 1 "Floppy-Power" H 1825 2175 50  0000 L CNN
 F 2 "floppy_power:Floppy_Power_1x04_Pitch2.54mm" H 1975 1925 50  0001 C CNN
@@
 P 1600 1925
 AR Path="/5CEBDDD4" Ref="#PWR?"  Part="1"
-AR Path="/5CD0EE48/5CEBDDD4" Ref="#PWR02"  Part="1"
-F 0 "#PWR02" H 1600 1675 50  0001 C CNN
+AR Path="/5CD0EE48/5CEBDDD4" Ref="#PWR011"  Part="1"
+F 0 "#PWR011" H 1600 1675 50  0001 C CNN
 F 1 "GND" H 1605 1752 50  0000 C CNN
 F 2 "" H 1600 1925 50  0001 C CNN
@@
 AR Path="/5D1F80E4" Ref="#PWR?"  Part="1"
 AR Path="/5CD1E0A5/5D1F80E4" Ref="#PWR?"  Part="1"
-AR Path="/5CD0EE48/5D1F80E4" Ref="#PWR03"  Part="1"
-F 0 "#PWR03" H 1975 2825 50  0001 C CNN
+AR Path="/5CD0EE48/5D1F80E4" Ref="#PWR012"  Part="1"
+F 0 "#PWR012" H 1975 2825 50  0001 C CNN
 F 1 "VCC" H 1992 3148 50  0000 C CNN
 F 2 "" H 1975 2975 50  0001 C CNN
@@
 AR Path="/5D1F80EA" Ref="#PWR?"  Part="1"
 AR Path="/5CD1E0A5/5D1F80EA" Ref="#PWR?"  Part="1"
-AR Path="/5CD0EE48/5D1F80EA" Ref="#PWR04"  Part="1"
-F 0 "#PWR04" H 2875 4125 50  0001 C CNN
+AR Path="/5CD0EE48/5D1F80EA" Ref="#PWR013"  Part="1"
+F 0 "#PWR013" H 2875 4125 50  0001 C CNN
 F 1 "GND" H 2880 4202 50  0000 C CNN
 F 2 "" H 2875 4375 50  0001 C CNN
@@
 AR Path="/5D1F80FB" Ref="#PWR?"  Part="1"
 AR Path="/5CD1E0A5/5D1F80FB" Ref="#PWR?"  Part="1"
-AR Path="/5CD0EE48/5D1F80FB" Ref="#PWR07"  Part="1"
-F 0 "#PWR07" H 4575 2575 50  0001 C CNN
+AR Path="/5CD0EE48/5D1F80FB" Ref="#PWR016"  Part="1"
+F 0 "#PWR016" H 4575 2575 50  0001 C CNN
 F 1 "VCC" H 4592 2898 50  0000 C CNN
 F 2 "" H 4575 2725 50  0001 C CNN
@@
 AR Path="/5D1F8101" Ref="#PWR?"  Part="1"
 AR Path="/5CD1E0A5/5D1F8101" Ref="#PWR?"  Part="1"
-AR Path="/5CD0EE48/5D1F8101" Ref="#PWR05"  Part="1"
-F 0 "#PWR05" H 3125 2600 50  0001 C CNN
+AR Path="/5CD0EE48/5D1F8101" Ref="#PWR014"  Part="1"
+F 0 "#PWR014" H 3125 2600 50  0001 C CNN
 F 1 "GND" H 3130 2677 50  0000 C CNN
 F 2 "" H 3125 2850 50  0001 C CNN
@@
 AR Path="/5D1F8117" Ref="#PWR?"  Part="1"
 AR Path="/5CD1E0A5/5D1F8117" Ref="#PWR?"  Part="1"
-AR Path="/5CD0EE48/5D1F8117" Ref="#PWR06"  Part="1"
-F 0 "#PWR06" H 3875 3725 50  0001 C CNN
+AR Path="/5CD0EE48/5D1F8117" Ref="#PWR015"  Part="1"
+F 0 "#PWR015" H 3875 3725 50  0001 C CNN
 F 1 "GND" H 3880 3802 50  0000 C CNN
 F 2 "" H 3875 3975 50  0001 C CNN

Commit message: pcb: assign footprints
Parts:
- J8: footprint Connector_PinHeader_2.54mm:PinHeader_2x17_P2.54mm_Horizontal -> Connector_PinHeader_2.54mm:PinHeader_2x17_P2.54mm_Vertical
- R1, R2, R3, R4, R5, R6: footprint (none) -> Capacitor_SMD:C_0201_0603Metric
- SW1: footprint Buttons_Switches_THT:SW_DIP_x6_W7.62mm_Slide -> Button_Switch_THT:SW_DIP_SPSTx06_Slide_9.78x17.42mm_W7.62mm_P2.54mm
- U1: footprint (none) -> Package_DIP:DIP-16_W7.62mm
Changed lines of the file:
@@
 $Descr A4 11693 8268
 encoding utf-8
-Sheet 5 6
+Sheet 4 6
 Title ""
 Date ""
@@
 F 0 "J8" H 7075 4475 50  0000 C CNN
 F 1 "IBM_PC_Floppy_IDC" H 7125 4375 50  0000 C CNN
-F 2 "Connector_PinHeader_2.54mm:PinHeader_2x17_P2.54mm_Horizontal" H 6875 3425 50  0001 C CNN
+F 2 "Connector_PinHeader_2.54mm:PinHeader_2x17_P2.54mm_Vertical" H 6875 3425 50  0001 C CNN
 F 3 "" H 6875 3425 50  0001 C CNN
 	1    6875 3425
@@
 F 0 "SW1" H 2275 3925 50  0000 C CNN
 F 1 "Bus Address Select" H 2275 3125 50  0000 C CNN
-F 2 "Buttons_Switches_THT:SW_DIP_x6_W7.62mm_Slide" H 2275 3475 50  0001 C CNN
+F 2 "Button_Switch_THT:SW_DIP_SPSTx06_Slide_9.78x17.42mm_W7.62mm_P2.54mm" H 2275 3475 50  0001 C CNN
 F 3 "" H 2275 3475 50  0001 C CNN
 	1    2275 3475
@@
 F 0 "R6" V 3425 3575 50  0000 L CNN
 F 1 "4K7" V 3375 3800 50  0000 L CNN
-F 2 "" V 3305 3875 50  0001 C CNN
+F 2 "Capacitor_SMD:C_0201_0603Metric" V 3305 3875 50  0001 C CNN
 F 3 "~" H 3375 3875 50  0001 C CNN
 	1    3375 3875
@@
 F 0 "R5" V 3325 3575 50  0000 L CNN
 F 1 "4K7" V 3275 3800 50  0000 L CNN
-F 2 "" V 3205 3875 50  0001 C CNN
+F 2 "Capacitor_SMD:C_0201_0603Metric" V 3205 3875 50  0001 C CNN
 F 3 "~" H 3275 3875 50  0001 C CNN
 	1    3275 3875
@@
 F 0 "R4" V 3225 3575 50  0000 L CNN
 F 1 "4K7" V 3175 3800 50  0000 L CNN
-F 2 "" V 3105 3875 50  0001 C CNN
+F 2 "Capacitor_SMD:C_0201_0603Metric" V 3105 3875 50  0001 C CNN
 F 3 "~" H 3175 3875 50  0001 C CNN
 	1    3175 3875
@@
 F 0 "R3" V 3125 3575 50  0000 L CNN
 F 1 "4K7" V 3075 3800 50  0000 L CNN
-F 2 "" V 3005 3875 50  0001 C CNN
+F 2 "Capacitor_SMD:C_0201_0603Metric" V 3005 3875 50  0001 C CNN
 F 3 "~" H 3075 3875 50  0001 C CNN
 	1    3075 3875
@@
 F 0 "R2" V 3025 3575 50  0000 L CNN
 F 1 "4K7" V 2975 3800 50  0000 L CNN
-F 2 "" V 2905 3875 50  0001 C CNN
+F 2 "Capacitor_SMD:C_0201_0603Metric" V 2905 3875 50  0001 C CNN
 F 3 "~" H 2975 3875 50  0001 C CNN
 	1    2975 3875
@@
 F 0 "R1" V 2925 3575 50  0000 L CNN
 F 1 "4K7" V 2875 3800 50  0000 L CNN
-F 2 "" V 2805 3875 50  0001 C CNN
+F 2 "Capacitor_SMD:C_0201_0603Metric" V 2805 3875 50  0001 C CNN
 F 3 "~" H 2875 3875 50  0001 C CNN
 	1    2875 3875
@@
 F 0 "U1" H 4275 3650 50  0000 C CNN
 F 1 "4021" H 4275 3550 50  0000 C CNN
-F 2 "" H 4425 3125 50  0001 C CNN
+F 2 "Package_DIP:DIP-16_W7.62mm" H 4425 3125 50  0001 C CNN
 F 3 "" H 4425 3125 50  0001 C CNN
 	1    4425 3125

Commit message: pcb: add I2C eeprom
Parts:
- J8: footprint Connector_PinHeader_2.54mm:PinHeader_2x17_P2.54mm_Vertical -> Connector_PinHeader_2.54mm:PinHeader_2x17_P2.54mm_Horizontal
- U1: footprint Package_DIP:DIP-16_W7.62mm -> Package_SO:SSOP-16_5.3x6.2mm_P0.65mm
Changed lines of the file:
@@
 F 0 "J8" H 7075 4475 50  0000 C CNN
 F 1 "IBM_PC_Floppy_IDC" H 7125 4375 50  0000 C CNN
-F 2 "Connector_PinHeader_2.54mm:PinHeader_2x17_P2.54mm_Vertical" H 6875 3425 50  0001 C CNN
+F 2 "Connector_PinHeader_2.54mm:PinHeader_2x17_P2.54mm_Horizontal" H 6875 3425 50  0001 C CNN
 F 3 "" H 6875 3425 50  0001 C CNN
 	1    6875 3425
@@
 P 7075 4425
 AR Path="/5CE2645F" Ref="#PWR?"  Part="1"
-AR Path="/5CD0EE48/5CE2645F" Ref="#PWR017"  Part="1"
-F 0 "#PWR017" H 7075 4175 50  0001 C CNN
+AR Path="/5CD0EE48/5CE2645F" Ref="#PWR016"  Part="1"
+F 0 "#PWR016" H 7075 4175 50  0001 C CNN
 F 1 "GND" H 7080 4252 50  0000 C CNN
 F 2 "" H 7075 4425 50  0001 C CNN
@@
 P 1600 1925
 AR Path="/5CEBDDD4" Ref="#PWR?"  Part="1"
-AR Path="/5CD0EE48/5CEBDDD4" Ref="#PWR011"  Part="1"
-F 0 "#PWR011" H 1600 1675 50  0001 C CNN
+AR Path="/5CD0EE48/5CEBDDD4" Ref="#PWR010"  Part="1"
+F 0 "#PWR010" H 1600 1675 50  0001 C CNN
 F 1 "GND" H 1605 1752 50  0000 C CNN
 F 2 "" H 1600 1925 50  0001 C CNN
@@
 AR Path="/5D1F80E4" Ref="#PWR?"  Part="1"
 AR Path="/5CD1E0A5/5D1F80E4" Ref="#PWR?"  Part="1"
-AR Path="/5CD0EE48/5D1F80E4" Ref="#PWR012"  Part="1"
-F 0 "#PWR012" H 1975 2825 50  0001 C CNN
+AR Path="/5CD0EE48/5D1F80E4" Ref="#PWR011"  Part="1"
+F 0 "#PWR011" H 1975 2825 50  0001 C CNN
 F 1 "VCC" H 1992 3148 50  0000 C CNN
 F 2 "" H 1975 2975 50  0001 C CNN
@@
 AR Path="/5D1F80EA" Ref="#PWR?"  Part="1"
 AR Path="/5CD1E0A5/5D1F80EA" Ref="#PWR?"  Part="1"
-AR Path="/5CD0EE48/5D1F80EA" Ref="#PWR013"  Part="1"
-F 0 "#PWR013" H 2875 4125 50  0001 C CNN
+AR Path="/5CD0EE48/5D1F80EA" Ref="#PWR012"  Part="1"
+F 0 "#PWR012" H 2875 4125 50  0001 C CNN
 F 1 "GND" H 2880 4202 50  0000 C CNN
 F 2 "" H 2875 4375 50  0001 C CNN
@@
 AR Path="/5D1F80FB" Ref="#PWR?"  Part="1"
 AR Path="/5CD1E0A5/5D1F80FB" Ref="#PWR?"  Part="1"
-AR Path="/5CD0EE48/5D1F80FB" Ref="#PWR016"  Part="1"
-F 0 "#PWR016" H 4575 2575 50  0001 C CNN
+AR Path="/5CD0EE48/5D1F80FB" Ref="#PWR015"  Part="1"
+F 0 "#PWR015" H 4575 2575 50  0001 C CNN
 F 1 "VCC" H 4592 2898 50  0000 C CNN
 F 2 "" H 4575 2725 50  0001 C CNN
@@
 AR Path="/5D1F8101" Ref="#PWR?"  Part="1"
 AR Path="/5CD1E0A5/5D1F8101" Ref="#PWR?"  Part="1"
-AR Path="/5CD0EE48/5D1F8101" Ref="#PWR014"  Part="1"
-F 0 "#PWR014" H 3125 2600 50  0001 C CNN
+AR Path="/5CD0EE48/5D1F8101" Ref="#PWR013"  Part="1"
+F 0 "#PWR013" H 3125 2600 50  0001 C CNN
 F 1 "GND" H 3130 2677 50  0000 C CNN
 F 2 "" H 3125 2850 50  0001 C CNN
@@
 F 0 "U1" H 4275 3650 50  0000 C CNN
 F 1 "4021" H 4275 3550 50  0000 C CNN
-F 2 "Package_DIP:DIP-16_W7.62mm" H 4425 3125 50  0001 C CNN
+F 2 "Package_SO:SSOP-16_5.3x6.2mm_P0.65mm" H 4425 3125 50  0001 C CNN
 F 3 "" H 4425 3125 50  0001 C CNN
 	1    4425 3125
@@
 AR Path="/5D1F8117" Ref="#PWR?"  Part="1"
 AR Path="/5CD1E0A5/5D1F8117" Ref="#PWR?"  Part="1"
-AR Path="/5CD0EE48/5D1F8117" Ref="#PWR015"  Part="1"
-F 0 "#PWR015" H 3875 3725 50  0001 C CNN
+AR Path="/5CD0EE48/5D1F8117" Ref="#PWR014"  Part="1"
+F 0 "#PWR014" H 3875 3725 50  0001 C CNN
 F 1 "GND" H 3880 3802 50  0000 C CNN
 F 2 "" H 3875 3975 50  0001 C CNN

Commit message: pcb: continue placement + add some info on silk
Parts:
- added C2: 100nF, Capacitor_SMD:C_0805_2012Metric, symbol Device:C
- J8: footprint Connector_PinHeader_2.54mm:PinHeader_2x17_P2.54mm_Horizontal -> Connector_PinSocket_2.54mm:PinSocket_2x17_P2.54mm_Horizontal
- R1, R2, R3, R4, R5, R6: footprint Capacitor_SMD:C_0201_0603Metric -> Resistor_SMD:R_0805_2012Metric
Connections:
- net GND: now also C2.2
- net VCC: now also C2.1
Other:
- note added: "Bypass"
Changed lines of the file:
@@
 F 0 "J8" H 7075 4475 50  0000 C CNN
 F 1 "IBM_PC_Floppy_IDC" H 7125 4375 50  0000 C CNN
-F 2 "Connector_PinHeader_2.54mm:PinHeader_2x17_P2.54mm_Horizontal" H 6875 3425 50  0001 C CNN
+F 2 "Connector_PinSocket_2.54mm:PinSocket_2x17_P2.54mm_Horizontal" H 6875 3425 50  0001 C CNN
 F 3 "" H 6875 3425 50  0001 C CNN
 	1    6875 3425
@@
 P 7075 4425
 AR Path="/5CE2645F" Ref="#PWR?"  Part="1"
-AR Path="/5CD0EE48/5CE2645F" Ref="#PWR016"  Part="1"
-F 0 "#PWR016" H 7075 4175 50  0001 C CNN
+AR Path="/5CD0EE48/5CE2645F" Ref="#PWR018"  Part="1"
+F 0 "#PWR018" H 7075 4175 50  0001 C CNN
 F 1 "GND" H 7080 4252 50  0000 C CNN
 F 2 "" H 7075 4425 50  0001 C CNN
@@
 F 0 "R6" V 3425 3575 50  0000 L CNN
 F 1 "4K7" V 3375 3800 50  0000 L CNN
-F 2 "Capacitor_SMD:C_0201_0603Metric" V 3305 3875 50  0001 C CNN
+F 2 "Resistor_SMD:R_0805_2012Metric" V 3305 3875 50  0001 C CNN
 F 3 "~" H 3375 3875 50  0001 C CNN
 	1    3375 3875
@@
 F 0 "R5" V 3325 3575 50  0000 L CNN
 F 1 "4K7" V 3275 3800 50  0000 L CNN
-F 2 "Capacitor_SMD:C_0201_0603Metric" V 3205 3875 50  0001 C CNN
+F 2 "Resistor_SMD:R_0805_2012Metric" V 3205 3875 50  0001 C CNN
 F 3 "~" H 3275 3875 50  0001 C CNN
 	1    3275 3875
@@
 F 0 "R4" V 3225 3575 50  0000 L CNN
 F 1 "4K7" V 3175 3800 50  0000 L CNN
-F 2 "Capacitor_SMD:C_0201_0603Metric" V 3105 3875 50  0001 C CNN
+F 2 "Resistor_SMD:R_0805_2012Metric" V 3105 3875 50  0001 C CNN
 F 3 "~" H 3175 3875 50  0001 C CNN
 	1    3175 3875
@@
 F 0 "R3" V 3125 3575 50  0000 L CNN
 F 1 "4K7" V 3075 3800 50  0000 L CNN
-F 2 "Capacitor_SMD:C_0201_0603Metric" V 3005 3875 50  0001 C CNN
+F 2 "Resistor_SMD:R_0805_2012Metric" V 3005 3875 50  0001 C CNN
 F 3 "~" H 3075 3875 50  0001 C CNN
 	1    3075 3875
@@
 F 0 "R2" V 3025 3575 50  0000 L CNN
 F 1 "4K7" V 2975 3800 50  0000 L CNN
-F 2 "Capacitor_SMD:C_0201_0603Metric" V 2905 3875 50  0001 C CNN
+F 2 "Resistor_SMD:R_0805_2012Metric" V 2905 3875 50  0001 C CNN
 F 3 "~" H 2975 3875 50  0001 C CNN
 	1    2975 3875
@@
 F 0 "R1" V 2925 3575 50  0000 L CNN
 F 1 "4K7" V 2875 3800 50  0000 L CNN
-F 2 "Capacitor_SMD:C_0201_0603Metric" V 2805 3875 50  0001 C CNN
+F 2 "Resistor_SMD:R_0805_2012Metric" V 2805 3875 50  0001 C CNN
 F 3 "~" H 2875 3875 50  0001 C CNN
 	1    2875 3875
@@
 AR Path="/5D1F80FB" Ref="#PWR?"  Part="1"
 AR Path="/5CD1E0A5/5D1F80FB" Ref="#PWR?"  Part="1"
-AR Path="/5CD0EE48/5D1F80FB" Ref="#PWR015"  Part="1"
-F 0 "#PWR015" H 4575 2575 50  0001 C CNN
+AR Path="/5CD0EE48/5D1F80FB" Ref="#PWR017"  Part="1"
+F 0 "#PWR017" H 4575 2575 50  0001 C CNN
 F 1 "VCC" H 4592 2898 50  0000 C CNN
 F 2 "" H 4575 2725 50  0001 C CNN
@@
 AR Path="/5D1F8117" Ref="#PWR?"  Part="1"
 AR Path="/5CD1E0A5/5D1F8117" Ref="#PWR?"  Part="1"
-AR Path="/5CD0EE48/5D1F8117" Ref="#PWR014"  Part="1"
-F 0 "#PWR014" H 3875 3725 50  0001 C CNN
+AR Path="/5CD0EE48/5D1F8117" Ref="#PWR016"  Part="1"
+F 0 "#PWR016" H 3875 3725 50  0001 C CNN
 F 1 "GND" H 3880 3802 50  0000 C CNN
 F 2 "" H 3875 3975 50  0001 C CNN
@@
 Text HLabel 4975 3875 2    50   Output ~ 0
 MISO
+$Comp
+L Device:C C?
+U 1 1 5CD16AEF
+P 3300 1725
+AR Path="/5CD16AEF" Ref="C?"  Part="1"
+AR Path="/5CCFEC3E/5CD16AEF" Ref="C?"  Part="1"
+AR Path="/5CD1E0A5/5CD16AEF" Ref="C?"  Part="1"
+AR Path="/5CD0EE48/5CD16AEF" Ref="C2"  Part="1"
+F 0 "C2" H 3075 1925 50  0000 L CNN
+F 1 "100nF" H 3025 1825 50  0000 L CNN
+F 2 "Capacitor_SMD:C_0805_2012Metric" H 3338 1575 50  0001 C CNN
+F 3 "~" H 3300 1725 50  0001 C CNN
+	1    3300 1725
+	1    0    0    -1
+$EndComp
+$Comp
+L power:VCC #PWR?
+U 1 1 5CD16AF5
+P 3300 1450
+AR Path="/5CCFEC3E/5CD16AF5" Ref="#PWR?"  Part="1"
+AR Path="/5CD1E0A5/5CD16AF5" Ref="#PWR?"  Part="1"
+AR Path="/5CD0EE48/5CD16AF5" Ref="#PWR014"  Part="1"
+F 0 "#PWR014" H 3300 1300 50  0001 C CNN
+F 1 "VCC" H 3317 1623 50  0000 C CNN
+F 2 "" H 3300 1450 50  0001 C CNN
+F 3 "" H 3300 1450 50  0001 C CNN
+	1    3300 1450
+	1    0    0    -1
+$EndComp
+$Comp
+L power:GND #PWR?
+U 1 1 5CD16AFB
+P 3300 1975
+AR Path="/5CCFEC3E/5CD16AFB" Ref="#PWR?"  Part="1"
+AR Path="/5CD1E0A5/5CD16AFB" Ref="#PWR?"  Part="1"
+AR Path="/5CD0EE48/5CD16AFB" Ref="#PWR015"  Part="1"
+F 0 "#PWR015" H 3300 1725 50  0001 C CNN
+F 1 "GND" H 3305 1802 50  0000 C CNN
+F 2 "" H 3300 1975 50  0001 C CNN
+F 3 "" H 3300 1975 50  0001 C CNN
+	1    3300 1975
+	1    0    0    -1
+$EndComp
+Wire Wire Line
+	3300 1450 3300 1575
+Wire Wire Line
+	3300 1875 3300 1975
+Text Notes 2925 1400 0    50   ~ 0
+Bypass
 $EndSCHEMATC

Commit message: pcb: fix FTDI and floppy connector orientation
Parts:
- J8: footprint Connector_PinSocket_2.54mm:PinSocket_2x17_P2.54mm_Horizontal -> ibm_idc_floppy_connector:ibm_pc_floppy_idc
Changed lines of the file:
@@
 EESchema Schematic File Version 4
+LIBS:floppyorgel-cache
 EELAYER 29 0
 EELAYER END
@@
 F 0 "J8" H 7075 4475 50  0000 C CNN
 F 1 "IBM_PC_Floppy_IDC" H 7125 4375 50  0000 C CNN
-F 2 "Connector_PinSocket_2.54mm:PinSocket_2x17_P2.54mm_Horizontal" H 6875 3425 50  0001 C CNN
+F 2 "ibm_idc_floppy_connector:ibm_pc_floppy_idc" H 6875 3425 50  0001 C CNN
 F 3 "" H 6875 3425 50  0001 C CNN
 	1    6875 3425
