File: Arduino/pcb/bus.sch (KiCad schematic (older format))
At the start: 6 parts, among them J2 Floppy-Bus, J3 MAX485 Socket, J4 Floppy-Bus

Commit message: pcb: reannotate symbols
Parts:
- renumbered C1 to C6, J3 to J6, J2 to J7, J4 to J8, R1 to R15, R2 to R16
Changed lines of the file:
@@
 $EndDescr
 $Comp
-L Interface_UART:MAX485E J3
+L Interface_UART:MAX485E J6
 U 1 1 5CF1EB96
 P 4875 1575
-F 0 "J3" H 4500 2175 50  0000 C CNN
+F 0 "J6" H 4500 2175 50  0000 C CNN
 F 1 "MAX485 Socket" H 4475 2075 50  0000 C CNN
 F 2 "dil:dil_8-300_socket" H 4875 1575 50  0001 C CNN
@@
 $EndComp
 $Comp
-L power:VCC #PWR04
+L power:VCC #PWR030
 U 1 1 5CF1EBBB
 P 4875 975
-F 0 "#PWR04" H 4875 825 50  0001 C CNN
+F 0 "#PWR030" H 4875 825 50  0001 C CNN
 F 1 "VCC" H 4892 1148 50  0000 C CNN
 F 2 "" H 4875 975 50  0001 C CNN
@@
 $EndComp
 $Comp
-L power:GND #PWR05
+L power:GND #PWR031
 U 1 1 5CF1EBC1
 P 4875 2275
-F 0 "#PWR05" H 4875 2025 50  0001 C CNN
+F 0 "#PWR031" H 4875 2025 50  0001 C CNN
 F 1 "GND" H 4880 2102 50  0000 C CNN
 F 2 "" H 4875 2275 50  0001 C CNN
@@
 AR Path="/5D17F33C" Ref="C?"  Part="1"
 AR Path="/5CCFEC3E/5D17F33C" Ref="C?"  Part="1"
-AR Path="/5CD1E0A5/5D17F33C" Ref="C1"  Part="1"
-F 0 "C1" H 3700 1800 50  0000 L CNN
+AR Path="/5CD1E0A5/5D17F33C" Ref="C6"  Part="1"
+F 0 "C6" H 3700 1800 50  0000 L CNN
 F 1 "100nF" H 3650 1700 50  0000 L CNN
 F 2 "Capacitor_SMD:C_0805_2012Metric" H 3963 1450 50  0001 C CNN
@@
 P 3925 1325
 AR Path="/5CCFEC3E/5D17F342" Ref="#PWR?"  Part="1"
-AR Path="/5CD1E0A5/5D17F342" Ref="#PWR02"  Part="1"
-F 0 "#PWR02" H 3925 1175 50  0001 C CNN
+AR Path="/5CD1E0A5/5D17F342" Ref="#PWR028"  Part="1"
+F 0 "#PWR028" H 3925 1175 50  0001 C CNN
 F 1 "VCC" H 3942 1498 50  0000 C CNN
 F 2 "" H 3925 1325 50  0001 C CNN
@@
 P 3925 1850
 AR Path="/5CCFEC3E/5D17F348" Ref="#PWR?"  Part="1"
-AR Path="/5CD1E0A5/5D17F348" Ref="#PWR03"  Part="1"
-F 0 "#PWR03" H 3925 1600 50  0001 C CNN
+AR Path="/5CD1E0A5/5D17F348" Ref="#PWR029"  Part="1"
+F 0 "#PWR029" H 3925 1600 50  0001 C CNN
 F 1 "GND" H 3930 1677 50  0000 C CNN
 F 2 "" H 3925 1850 50  0001 C CNN
@@
 Bypass
 $Comp
-L power:PWR_FLAG #FLG01
+L power:PWR_FLAG #FLG02
 U 1 1 5D1B34B5
 P 10800 1200
-F 0 "#FLG01" H 10800 1275 50  0001 C CNN
+F 0 "#FLG02" H 10800 1275 50  0001 C CNN
 F 1 "PWR_FLAG" H 10800 1373 50  0000 C CNN
 F 2 "" H 10800 1200 50  0001 C CNN
@@
 Connection ~ 10800 1300
 $Comp
-L floppy-bus-connector:Floppy-Bus J4
+L floppy-bus-connector:Floppy-Bus J8
 U 1 1 5D1ABE61
 P 9050 1425
-F 0 "J4" H 9250 1842 50  0000 C CNN
+F 0 "J8" H 9250 1842 50  0000 C CNN
 F 1 "Floppy-Bus" H 9250 1751 50  0000 C CNN
 F 2 "shrouded:Shrouded_Header_2x05_Pitch2.54mm" H 9050 1425 50  0001 C CNN
@@
 20V
 $Comp
-L power:GND #PWR06
+L power:GND #PWR034
 U 1 1 5CDB5675
 P 10625 1900
-F 0 "#PWR06" H 10625 1650 50  0001 C CNN
+F 0 "#PWR034" H 10625 1650 50  0001 C CNN
 F 1 "GND" H 10630 1727 50  0000 C CNN
 F 2 "" H 10625 1900 50  0001 C CNN
@@
 GND
 $Comp
-L floppy-bus-connector:Floppy-Bus J2
+L floppy-bus-connector:Floppy-Bus J7
 U 1 1 5D1AADEF
 P 7550 1425
-F 0 "J2" H 7750 1842 50  0000 C CNN
+F 0 "J7" H 7750 1842 50  0000 C CNN
 F 1 "Floppy-Bus" H 7750 1751 50  0000 C CNN
 F 2 "shrouded:Shrouded_Header_2x05_Pitch2.54mm" H 7550 1425 50  0001 C CNN
@@
 BUS_TX_EN
 $Comp
-L Device:R R1
+L Device:R R15
 U 1 1 5D9A9AF7
 P 5975 1325
-F 0 "R1" H 6045 1371 50  0000 L CNN
+F 0 "R15" H 6045 1371 50  0000 L CNN
 F 1 "4k7" V 5975 1250 50  0000 L CNN
 F 2 "Resistor_SMD:R_0805_2012Metric" V 5905 1325 50  0001 C CNN
@@
 $EndComp
 $Comp
-L Device:R R2
+L Device:R R16
 U 1 1 5D9A9F68
 P 5975 1925
-F 0 "R2" H 6045 1971 50  0000 L CNN
+F 0 "R16" H 6045 1971 50  0000 L CNN
 F 1 "4k7" V 5975 1850 50  0000 L CNN
 F 2 "Resistor_SMD:R_0805_2012Metric" V 5905 1925 50  0001 C CNN
@@
 Connection ~ 5975 1675
 $Comp
-L power:VCC #PWR0105
+L power:VCC #PWR032
 U 1 1 5D9C25C7
 P 5975 975
-F 0 "#PWR0105" H 5975 825 50  0001 C CNN
+F 0 "#PWR032" H 5975 825 50  0001 C CNN
 F 1 "VCC" H 5992 1148 50  0000 C CNN
 F 2 "" H 5975 975 50  0001 C CNN
@@
 $EndComp
 $Comp
-L power:GND #PWR0106
+L power:GND #PWR033
 U 1 1 5D9C302F
 P 5975 2275
-F 0 "#PWR0106" H 5975 2025 50  0001 C CNN
+F 0 "#PWR033" H 5975 2025 50  0001 C CNN
 F 1 "GND" H 5980 2102 50  0000 C CNN
 F 2 "" H 5975 2275 50  0001 C CNN
