File: Arduino/pcb/power.sch (KiCad schematic (older format))
At the start: 0 parts

Commit message: pcb: continue wiring / move parts to hierachival sheets
Parts:
- added C3: 1500uF, symbol Device:CP
- added J7: Buck-Converter-5V, symbol buck-converter:Buck-Converter
- added J8: Buck-Converter-12V, symbol buck-converter:Buck-Converter
Connections:
- new net 12V_BUS: J8.4 (Pin_4)
- new net 5V_BUS: J7.4 (Pin_4)
- new net BUS_POWER: C3.1, J7.1 (Pin_1), J7.2 (Pin_2), J8.1 (Pin_1), J8.2 (Pin_2)
- new net GND: C3.2, J7.3 (Pin_3), J8.3 (Pin_3)
Changed lines of the file:
@@
 $Descr A4 11693 8268
 encoding utf-8
-Sheet 1 6
+Sheet 4 6
 Title ""
 Date ""
@@
 Comment4 ""
 $EndDescr
+$Comp
+L Device:CP C?
+U 1 1 5CFDD059
+P 3425 4625
+AR Path="/5CFDD059" Ref="C?"  Part="1"
+AR Path="/5CD31258/5CFDD059" Ref="C3"  Part="1"
+F 0 "C3" H 3543 4671 50  0000 L CNN
+F 1 "1500uF" H 3543 4580 50  0000 L CNN
+F 2 "" H 3463 4475 50  0001 C CNN
+F 3 "~" H 3425 4625 50  0001 C CNN
+	1    3425 4625
+	1    0    0    -1
+$EndComp
+$Comp
+L power:GND #PWR?
+U 1 1 5CFDD061
+P 3425 4775
+AR Path="/5CFDD061" Ref="#PWR?"  Part="1"
+AR Path="/5CD31258/5CFDD061" Ref="#PWR015"  Part="1"
+F 0 "#PWR015" H 3425 4525 50  0001 C CNN
+F 1 "GND" H 3430 4602 50  0000 C CNN
+F 2 "" H 3425 4775 50  0001 C CNN
+F 3 "" H 3425 4775 50  0001 C CNN
+	1    3425 4775
+	1    0    0    -1
+$EndComp
+Wire Wire Line
+	4175 3725 4175 3825
+Wire Wire Line
+	4175 4025 4175 4175
+Wire Wire Line
+	4175 3825 3925 3825
+Connection ~ 4175 4650
+Wire Wire Line
+	4175 4550 4175 4650
+Wire Wire Line
+	4175 4650 3925 4650
+$Comp
+L power:GND #PWR?
+U 1 1 5CFDD037
+P 4050 4750
+AR Path="/5CFDD037" Ref="#PWR?"  Part="1"
+AR Path="/5CD31258/5CFDD037" Ref="#PWR017"  Part="1"
+F 0 "#PWR017" H 4050 4500 50  0001 C CNN
+F 1 "GND" H 4055 4577 50  0000 C CNN
+F 2 "" H 4050 4750 50  0001 C CNN
+F 3 "" H 4050 4750 50  0001 C CNN
+	1    4050 4750
+	1    0    0    -1
+$EndComp
+Text HLabel 3200 4225 0    50   Input ~ 0
+BUS_POWER
+Wire Wire Line
+	4175 4175 4275 4175
+Wire Wire Line
+	4175 4850 4175 5000
+Wire Wire Line
+	4175 5000 4300 5000
+$Comp
+L power:GND #PWR016
+U 1 1 5D0DAB46
+P 4050 3925
+F 0 "#PWR016" H 4050 3675 50  0001 C CNN
+F 1 "GND" H 4055 3752 50  0000 C CNN
+F 2 "" H 4050 3925 50  0001 C CNN
+F 3 "" H 4050 3925 50  0001 C CNN
+	1    4050 3925
+	1    0    0    -1
+$EndComp
+Wire Wire Line
+	4175 3925 4050 3925
+Wire Wire Line
+	4175 4750 4050 4750
+Text HLabel 4300 5000 2    50   Output ~ 0
+12V_BUS
+Wire Wire Line
+	3200 4225 3425 4225
+Wire Wire Line
+	3425 4475 3425 4225
+Connection ~ 3425 4225
+Wire Wire Line
+	3425 4225 3925 4225
+Connection ~ 3925 4225
+Wire Wire Line
+	3925 4225 3925 4650
+Wire Wire Line
+	3925 3825 3925 4225
+Text HLabel 4275 4175 2    50   Output ~ 0
+5V_BUS
+$Comp
+L buck-converter:Buck-Converter J8
+U 1 1 5D19DC09
+P 4375 4650
+F 0 "J8" H 4605 4642 50  0000 L CNN
+F 1 "Buck-Converter-12V" H 4605 4551 50  0000 L CNN
+F 2 "" H 4375 4650 50  0001 C CNN
+F 3 "" H 4375 4650 50  0001 C CNN
+	1    4375 4650
+	1    0    0    -1
+$EndComp
+$Comp
+L buck-converter:Buck-Converter J7
+U 1 1 5D19E626
+P 4375 3825
+F 0 "J7" H 4605 3817 50  0000 L CNN
+F 1 "Buck-Converter-5V" H 4605 3726 50  0000 L CNN
+F 2 "" H 4375 3825 50  0001 C CNN
+F 3 "" H 4375 3825 50  0001 C CNN
+	1    4375 3825
+	1    0    0    -1
+$EndComp
+Connection ~ 4175 3825
 $EndSCHEMATC

Commit message: pcb: finish wiring / use ws2812 under chip led
Parts:
- renumbered J7 to J5, J8 to J6
Changed lines of the file:
@@
 $Descr A4 11693 8268
 encoding utf-8
-Sheet 4 6
+Sheet 3 6
 Title ""
 Date ""
@@
 P 3425 4775
 AR Path="/5CFDD061" Ref="#PWR?"  Part="1"
-AR Path="/5CD31258/5CFDD061" Ref="#PWR015"  Part="1"
-F 0 "#PWR015" H 3425 4525 50  0001 C CNN
+AR Path="/5CD31258/5CFDD061" Ref="#PWR08"  Part="1"
+F 0 "#PWR08" H 3425 4525 50  0001 C CNN
 F 1 "GND" H 3430 4602 50  0000 C CNN
 F 2 "" H 3425 4775 50  0001 C CNN
@@
 P 4050 4750
 AR Path="/5CFDD037" Ref="#PWR?"  Part="1"
-AR Path="/5CD31258/5CFDD037" Ref="#PWR017"  Part="1"
-F 0 "#PWR017" H 4050 4500 50  0001 C CNN
+AR Path="/5CD31258/5CFDD037" Ref="#PWR010"  Part="1"
+F 0 "#PWR010" H 4050 4500 50  0001 C CNN
 F 1 "GND" H 4055 4577 50  0000 C CNN
 F 2 "" H 4050 4750 50  0001 C CNN
@@
 	4175 5000 4300 5000
 $Comp
-L power:GND #PWR016
+L power:GND #PWR09
 U 1 1 5D0DAB46
 P 4050 3925
-F 0 "#PWR016" H 4050 3675 50  0001 C CNN
+F 0 "#PWR09" H 4050 3675 50  0001 C CNN
 F 1 "GND" H 4055 3752 50  0000 C CNN
 F 2 "" H 4050 3925 50  0001 C CNN
@@
 5V_BUS
 $Comp
-L buck-converter:Buck-Converter J8
+L buck-converter:Buck-Converter J6
 U 1 1 5D19DC09
 P 4375 4650
-F 0 "J8" H 4605 4642 50  0000 L CNN
+F 0 "J6" H 4605 4642 50  0000 L CNN
 F 1 "Buck-Converter-12V" H 4605 4551 50  0000 L CNN
 F 2 "" H 4375 4650 50  0001 C CNN
@@
 $EndComp
 $Comp
-L buck-converter:Buck-Converter J7
+L buck-converter:Buck-Converter J5
 U 1 1 5D19E626
 P 4375 3825
-F 0 "J7" H 4605 3817 50  0000 L CNN
+F 0 "J5" H 4605 3817 50  0000 L CNN
 F 1 "Buck-Converter-5V" H 4605 3726 50  0000 L CNN
 F 2 "" H 4375 3825 50  0001 C CNN

Commit message: pcb: assign footprints
Parts:
- C3: footprint (none) -> Capacitor_THT:CP_Axial_L30.0mm_D18.0mm_P35.00mm_Horizontal
- J5, J6: footprint (none) -> Connector_PinSocket_2.54mm:PinSocket_1x04_P2.54mm_Vertical
Changed lines of the file:
@@
 F 0 "C3" H 3543 4671 50  0000 L CNN
 F 1 "1500uF" H 3543 4580 50  0000 L CNN
-F 2 "" H 3463 4475 50  0001 C CNN
+F 2 "Capacitor_THT:CP_Axial_L30.0mm_D18.0mm_P35.00mm_Horizontal" H 3463 4475 50  0001 C CNN
 F 3 "~" H 3425 4625 50  0001 C CNN
 	1    3425 4625
@@
 F 0 "J6" H 4605 4642 50  0000 L CNN
 F 1 "Buck-Converter-12V" H 4605 4551 50  0000 L CNN
-F 2 "" H 4375 4650 50  0001 C CNN
+F 2 "Connector_PinSocket_2.54mm:PinSocket_1x04_P2.54mm_Vertical" H 4375 4650 50  0001 C CNN
 F 3 "" H 4375 4650 50  0001 C CNN
 	1    4375 4650
@@
 F 0 "J5" H 4605 3817 50  0000 L CNN
 F 1 "Buck-Converter-5V" H 4605 3726 50  0000 L CNN
-F 2 "" H 4375 3825 50  0001 C CNN
+F 2 "Connector_PinSocket_2.54mm:PinSocket_1x04_P2.54mm_Vertical" H 4375 3825 50  0001 C CNN
 F 3 "" H 4375 3825 50  0001 C CNN
 	1    4375 3825

Commit message: pcb: add I2C eeprom
Parts:
- removed C3: 1500uF, Capacitor_THT:CP_Axial_L30.0mm_D18.0mm_P35.00mm_Horizontal, symbol Device:CP
Changed lines of the file:
@@
 Comment4 ""
 $EndDescr
-$Comp
-L Device:CP C?
-U 1 1 5CFDD059
-P 3425 4625
-AR Path="/5CFDD059" Ref="C?"  Part="1"
-AR Path="/5CD31258/5CFDD059" Ref="C3"  Part="1"
-F 0 "C3" H 3543 4671 50  0000 L CNN
-F 1 "1500uF" H 3543 4580 50  0000 L CNN
-F 2 "Capacitor_THT:CP_Axial_L30.0mm_D18.0mm_P35.00mm_Horizontal" H 3463 4475 50  0001 C CNN
-F 3 "~" H 3425 4625 50  0001 C CNN
-	1    3425 4625
-	1    0    0    -1
-$EndComp
-$Comp
-L power:GND #PWR?
-U 1 1 5CFDD061
-P 3425 4775
-AR Path="/5CFDD061" Ref="#PWR?"  Part="1"
-AR Path="/5CD31258/5CFDD061" Ref="#PWR08"  Part="1"
-F 0 "#PWR08" H 3425 4525 50  0001 C CNN
-F 1 "GND" H 3430 4602 50  0000 C CNN
-F 2 "" H 3425 4775 50  0001 C CNN
-F 3 "" H 3425 4775 50  0001 C CNN
-	1    3425 4775
-	1    0    0    -1
-$EndComp
 Wire Wire Line
 	4175 3725 4175 3825
@@
 P 4050 4750
 AR Path="/5CFDD037" Ref="#PWR?"  Part="1"
-AR Path="/5CD31258/5CFDD037" Ref="#PWR010"  Part="1"
-F 0 "#PWR010" H 4050 4500 50  0001 C CNN
+AR Path="/5CD31258/5CFDD037" Ref="#PWR09"  Part="1"
+F 0 "#PWR09" H 4050 4500 50  0001 C CNN
 F 1 "GND" H 4055 4577 50  0000 C CNN
 F 2 "" H 4050 4750 50  0001 C CNN
@@
 	4175 5000 4300 5000
 $Comp
-L power:GND #PWR09
+L power:GND #PWR08
 U 1 1 5D0DAB46
 P 4050 3925
-F 0 "#PWR09" H 4050 3675 50  0001 C CNN
+F 0 "#PWR08" H 4050 3675 50  0001 C CNN
 F 1 "GND" H 4055 3752 50  0000 C CNN
 F 2 "" H 4050 3925 50  0001 C CNN
@@
 Text HLabel 4300 5000 2    50   Output ~ 0
 12V_BUS
-Wire Wire Line
-	3200 4225 3425 4225
-Wire Wire Line
-	3425 4475 3425 4225
-Connection ~ 3425 4225
-Wire Wire Line
-	3425 4225 3925 4225
 Connection ~ 3925 4225
 Wire Wire Line
@@
 $EndComp
 Connection ~ 4175 3825
+Wire Wire Line
+	3200 4225 3925 4225
 $EndSCHEMATC

Commit message: pcb: reannotate symbols
Parts:
- renumbered J5 to J2, J6 to J3
Changed lines of the file:
@@
 P 4050 4750
 AR Path="/5CFDD037" Ref="#PWR?"  Part="1"
-AR Path="/5CD31258/5CFDD037" Ref="#PWR09"  Part="1"
-F 0 "#PWR09" H 4050 4500 50  0001 C CNN
+AR Path="/5CD31258/5CFDD037" Ref="#PWR03"  Part="1"
+F 0 "#PWR03" H 4050 4500 50  0001 C CNN
 F 1 "GND" H 4055 4577 50  0000 C CNN
 F 2 "" H 4050 4750 50  0001 C CNN
@@
 	4175 5000 4300 5000
 $Comp
-L power:GND #PWR08
+L power:GND #PWR02
 U 1 1 5D0DAB46
 P 4050 3925
-F 0 "#PWR08" H 4050 3675 50  0001 C CNN
+F 0 "#PWR02" H 4050 3675 50  0001 C CNN
 F 1 "GND" H 4055 3752 50  0000 C CNN
 F 2 "" H 4050 3925 50  0001 C CNN
@@
 5V_BUS
 $Comp
-L buck-converter:Buck-Converter J6
+L buck-converter:Buck-Converter J3
 U 1 1 5D19DC09
 P 4375 4650
-F 0 "J6" H 4605 4642 50  0000 L CNN
+F 0 "J3" H 4605 4642 50  0000 L CNN
 F 1 "Buck-Converter-12V" H 4605 4551 50  0000 L CNN
 F 2 "Connector_PinSocket_2.54mm:PinSocket_1x04_P2.54mm_Vertical" H 4375 4650 50  0001 C CNN
@@
 $EndComp
 $Comp
-L buck-converter:Buck-Converter J5
+L buck-converter:Buck-Converter J2
 U 1 1 5D19E626
 P 4375 3825
-F 0 "J5" H 4605 3817 50  0000 L CNN
+F 0 "J2" H 4605 3817 50  0000 L CNN
 F 1 "Buck-Converter-5V" H 4605 3726 50  0000 L CNN
 F 2 "Connector_PinSocket_2.54mm:PinSocket_1x04_P2.54mm_Vertical" H 4375 3825 50  0001 C CNN
